Commit message: add lidar

File: src/ppp_description/urdf/ppp.xacro (robot description, xacro)
@@ -367,4 +367,104 @@
   </collision>
 </link>
+<link name="forward_top_1_1">
+  <inertial>
+    <origin rpy="0 0 0" xyz="0.06502199144873529 -0.09472380566284748 0.0004895173930853369"/>
+    <mass value="0.48710215659029577"/>
+    <inertia ixx="0.00099" ixy="0.000235" ixz="1e-06" iyy="0.000784" iyz="-1e-06" izz="0.001773"/>
+  </inertial>
+  <visual>
+    <origin rpy="0 0 0" xyz="0.0 -0.149 -0.11"/>
+    <geometry>
+      <mesh filename="package://ppp_description/meshes/forward_top_1_1.stl" scale="0.001 0.001 0.001"/>
+    </geometry>
+    <material name="silver"/>
+  </visual>
+  <collision>
+    <origin rpy="0 0 0" xyz="0.0 -0.149 -0.11"/>
+    <geometry>
+      <mesh filename="package://ppp_description/meshes/forward_top_1_1.stl" scale="0.001 0.001 0.001"/>
+    </geometry>
+  </collision>
+</link>
+<link name="forward_top_1_Mirror__1">
+  <inertial>
+    <origin rpy="0 0 0" xyz="0.07845779784140774 0.07359181457392162 0.0004895171912021601"/>
+    <mass value="0.48710223650351714"/>
+    <inertia ixx="0.00099" ixy="-0.000234" ixz="-1e-06" iyy="0.000784" iyz="-1e-06" izz="0.001773"/>
+  </inertial>
+  <visual>
+    <origin rpy="0 0 0" xyz="0.14353 0.01936 -0.11"/>
+    <geometry>
+      <mesh filename="package://ppp_description/meshes/forward_top_1_Mirror__1.stl" scale="0.001 0.001 0.001"/>
+    </geometry>
+    <material name="silver"/>
+  </visual>
+  <collision>
+    <origin rpy="0 0 0" xyz="0.14353 0.01936 -0.11"/>
+    <geometry>
+      <mesh filename="package://ppp_description/meshes/forward_top_1_Mirror__1.stl" scale="0.001 0.001 0.001"/>
+    </geometry>
+  </collision>
+</link>
+<link name="back_top_1">
+  <inertial>
+    <origin rpy="0 0 0" xyz="0.07365321533839897 -0.06983833949014678 -0.0010887199497685018"/>
+    <mass value="0.23560428740017997"/>
+    <inertia ixx="0.00038" ixy="0.000345" ixz="1.8e-05" iyy="0.000537" iyz="-1.3e-05" izz="0.000907"/>
+  </inertial>
+  <visual>
+    <origin rpy="0 0 0" xyz="0.14353 0.01936 -0.11"/>
+    <geometry>
+      <mesh filename="package://ppp_description/meshes/back_top_1.stl" scale="0.001 0.001 0.001"/>
+    </geometry>
+    <material name="silver"/>
+  </visual>
+  <collision>
+    <origin rpy="0 0 0" xyz="0.14353 0.01936 -0.11"/>
+    <geometry>
+      <mesh filename="package://ppp_description/meshes/back_top_1.stl" scale="0.001 0.001 0.001"/>
+    </geometry>
+  </collision>
+</link>
+<link name="back_top2_1">
+  <inertial>
+    <origin rpy="0 0 0" xyz="-0.05499670719604889 -0.05870846160678311 0.0004968868769273244"/>
+    <mass value="0.18961170684744505"/>
+    <inertia ixx="0.000249" ixy="-0.000153" ixz="1e-06" iyy="0.000183" iyz="1e-06" izz="0.000432"/>
+  </inertial>
+  <visual>
+    <origin rpy="0 0 0" xyz="-0.14353 0.01936 -0.11"/>
+    <geometry>
+      <mesh filename="package://ppp_description/meshes/back_top2_1.stl" scale="0.001 0.001 0.001"/>
+    </geometry>
+    <material name="silver"/>
+  </visual>
+  <collision>
+    <origin rpy="0 0 0" xyz="-0.14353 0.01936 -0.11"/>
+    <geometry>
+      <mesh filename="package://ppp_description/meshes/back_top2_1.stl" scale="0.001 0.001 0.001"/>
+    </geometry>
+  </collision>
+</link>
+<link name="Lidar_1">
+  <inertial>
+    <origin rpy="0 0 0" xyz="1.0794814273332957e-07 2.1384410779645702e-07 0.03500000000000002"/>
+    <mass value="2.114723824855799"/>
+    <inertia ixx="0.001511" ixy="0.0" ixz="-0.0" iyy="0.001511" iyz="-0.0" izz="0.001295"/>
+  </inertial>
+  <visual>
+    <origin rpy="0 0 0" xyz="7.9e-05 -0.09632 -0.112"/>
+    <geometry>
+      <mesh filename="package://ppp_description/meshes/Lidar_1.stl" scale="0.001 0.001 0.001"/>
+    </geometry>
+    <material name="silver"/>
+  </visual>
+  <collision>
+    <origin rpy="0 0 0" xyz="7.9e-05 -0.09632 -0.112"/>
+    <geometry>
+      <mesh filename="package://ppp_description/meshes/Lidar_1.stl" scale="0.001 0.001 0.001"/>
+    </geometry>
+  </collision>
+</link>
 <joint name="Rev1" type="continuous">
   <origin rpy="0 0 0" xyz="0.04585 0.0 0.021125"/>
@@ -461,3 +561,28 @@
   <child link="IMU_1"/>
 </joint>
+<joint name="Rigid21" type="fixed">
+  <origin rpy="0 0 0" xyz="0.0 0.149 0.11"/>
+  <parent link="base_link"/>
+  <child link="forward_top_1_1"/>
+</joint>
+<joint name="Rigid22_1" type="fixed">
+  <origin rpy="0 0 0" xyz="-0.14353 -0.01936 0.11"/>
+  <parent link="base_link"/>
+  <child link="forward_top_1_Mirror__1"/>
+</joint>
+<joint name="Rigid23" type="fixed">
+  <origin rpy="0 0 0" xyz="-0.14353 -0.01936 0.11"/>
+  <parent link="base_link"/>
+  <child link="back_top_1"/>
+</joint>
+<joint name="Rigid24" type="fixed">
+  <origin rpy="0 0 0" xyz="0.14353 -0.01936 0.11"/>
+  <parent link="base_link"/>
+  <child link="back_top2_1"/>
+</joint>
+<joint name="Rigid25" type="fixed">
+  <origin rpy="0 0 0" xyz="0.143451 0.11568 0.002"/>
+  <parent link="forward_top_1_Mirror__1"/>
+  <child link="Lidar_1"/>
+</joint>
 </robot>

Commit message: fix lidar

File: src/ppp_description/urdf/ppp.xacro (robot description, xacro)
@@ -450,6 +450,6 @@
   <inertial>
     <origin rpy="0 0 0" xyz="1.0794814273332957e-07 2.1384410779645702e-07 0.03500000000000002"/>
-    <mass value="2.114723824855799"/>
-    <inertia ixx="0.001511" ixy="0.0" ixz="-0.0" iyy="0.001511" iyz="-0.0" izz="0.001295"/>
+    <mass value="0.0"/>
+    <inertia ixx="0.0" ixy="0.0" ixz="-0.0" iyy="0.0" iyz="-0.0" izz="0.0"/>
   </inertial>
   <visual>

Commit message: add diff drive

File: src/ppp_description/urdf/ppp.xacro (robot description, xacro)
@@ -472,5 +472,5 @@
   <child link="wheel_1"/>
   <axis xyz="1.0 0.0 -0.0"/>
-  <limit effort="10" velocity="100"/>
+  <!-- <limit effort="10" velocity="100"/> -->
 </joint>
 <joint name="Rev4" type="continuous">

Commit message: change ppp position yaw & change mapping launch

File: src/ppp_description/urdf/ppp.xacro (robot description, xacro)
@@ -6,10 +6,10 @@
 <link name="base_link">
   <inertial>
-    <origin rpy="0 0 0" xyz="1.5201671826907086e-05 -0.0012107786655712151 0.03300924453524418"/>
+    <origin rpy="0 0 1.5708" xyz="1.5201671826907086e-05 -0.0012107786655712151 0.03300924453524418"/>
     <mass value="4.737374361291242"/>
     <inertia ixx="0.040333" ixy="-5e-06" ixz="-1e-05" iyy="0.036454" iyz="0.001185" izz="0.066412"/>
   </inertial>
   <visual>
-    <origin rpy="0 0 0" xyz="0 0 0"/>
+    <origin rpy="0 0 1.5708" xyz="0 0 0"/>
     <geometry>
       <mesh filename="package://ppp_description/meshes/base_link.stl" scale="0.001 0.001 0.001"/>
@@ -18,5 +18,5 @@
   </visual>
   <collision>
-    <origin rpy="0 0 0" xyz="0 0 0"/>
+    <origin rpy="0 0 1.5708" xyz="0 0 0"/>
     <geometry>
       <mesh filename="package://ppp_description/meshes/base_link.stl" scale="0.001 0.001 0.001"/>

Commit message: fix launch hector

File: src/ppp_description/urdf/ppp.xacro (robot description, xacro)
@@ -5,11 +5,11 @@
 <xacro:include filename="$(find ppp_description)/urdf/ppp.gazebo" />
 <link name="base_link">
-  <inertial>
-    <origin rpy="0 0 1.5708" xyz="1.5201671826907086e-05 -0.0012107786655712151 0.03300924453524418"/>
+  <inertial><!--1.5708-->
+    <origin rpy="0 0 0" xyz="1.5201671826907086e-05 -0.0012107786655712151 0.03300924453524418"/>
     <mass value="4.737374361291242"/>
     <inertia ixx="0.040333" ixy="-5e-06" ixz="-1e-05" iyy="0.036454" iyz="0.001185" izz="0.066412"/>
   </inertial>
   <visual>
-    <origin rpy="0 0 1.5708" xyz="0 0 0"/>
+    <origin rpy="0 0 0" xyz="0 0 0"/>
     <geometry>
       <mesh filename="package://ppp_description/meshes/base_link.stl" scale="0.001 0.001 0.001"/>
@@ -18,5 +18,5 @@
   </visual>
   <collision>
-    <origin rpy="0 0 1.5708" xyz="0 0 0"/>
+    <origin rpy="0 0 0" xyz="0 0 0"/>
     <geometry>
       <mesh filename="package://ppp_description/meshes/base_link.stl" scale="0.001 0.001 0.001"/>
