Commit message: add correct urdf & debug settings & tf

File: src/ppp90_description/urdf/ppp90.xacro (robot description, xacro)
@@ -244,4 +244,24 @@
   </collision>
 </link>
+<link name="Forward_wheel_1">
+  <inertial>
+    <origin rpy="0 0 0" xyz="4.803445236845061e-07 -9.471071670506814e-08 -0.001437450709413722"/>
+    <mass value="0.0061871055650105375"/>
+    <inertia ixx="0.0" ixy="0.0" ixz="0.0" iyy="0.0" iyz="0.0" izz="1e-06"/>
+  </inertial>
+  <visual>
+    <origin rpy="0 0 0" xyz="0.120925 0.014338 -0.022"/>
+    <geometry>
+      <mesh filename="package://ppp90_description/meshes/Forward_wheel_1.stl" scale="0.001 0.001 0.001"/>
+    </geometry>
+    <material name="silver"/>
+  </visual>
+  <collision>
+    <origin rpy="0 0 0" xyz="0.120925 0.014338 -0.022"/>
+    <geometry>
+      <mesh filename="package://ppp90_description/meshes/Forward_wheel_1.stl" scale="0.001 0.001 0.001"/>
+    </geometry>
+  </collision>
+</link>
 <link name="forward_top_1_1">
   <inertial>
@@ -344,106 +364,4 @@
   </collision>
 </link>
-<!--FORWARD_WHEEL-->
-<link name="FW_baise_1">
-  <inertial>
-    <origin rpy="0 0 0" xyz="0.014149999999964021 -0.011650110353972745 -0.0014374507094137914"/>
-    <mass value="0.0061871055650105375"/>
-    <inertia ixx="0.0" ixy="0.0" ixz="-0.0" iyy="0.0" iyz="-0.0" izz="1e-06"/>
-  </inertial>
-  <visual>
-    <origin rpy="0 0 0" xyz="0.014 -0.117931 -0.022"/>
-    <geometry>
-      <mesh filename="package://ppp_description/meshes/FW_baise_1.stl" scale="0.001 0.001 0.001"/>
-    </geometry>
-    <material name="silver"/>
-  </visual>
-  <collision>
-    <origin rpy="0 0 0" xyz="0.014 -0.117931 -0.022"/>
-    <geometry>
-      <mesh filename="package://ppp_description/meshes/FW_baise_1.stl" scale="0.001 0.001 0.001"/>
-    </geometry>
-  </collision>
-</link>
-<link name="wheel__1__1">
-  <inertial>
-    <origin rpy="0 0 0" xyz="1.872807464664561e-14 -1.1035397273762015e-07 4.466912950640278e-17"/>
-    <mass value="0.0030771108424005812"/>
-    <inertia ixx="0.0" ixy="0.0" ixz="-0.0" iyy="0.0" iyz="-0.0" izz="0.0"/>
-  </inertial>
-  <visual>
-    <origin rpy="0 0 0" xyz="-0.00815 -0.106281 -0.0004"/>
-    <geometry>
-      <mesh filename="package://ppp_description/meshes/wheel__1__1.stl" scale="0.001 0.001 0.001"/>
-    </geometry>
-    <material name="silver"/>
-  </visual>
-  <collision>
-    <origin rpy="0 0 0" xyz="-0.00815 -0.106281 -0.0004"/>
-    <geometry>
-      <mesh filename="package://ppp_description/meshes/wheel__1__1.stl" scale="0.001 0.001 0.001"/>
-    </geometry>
-  </collision>
-</link>
-<link name="axis_1">
-  <inertial>
-    <origin rpy="0 0 0" xyz="0.03303899999968629 -1.1035397272374237e-07 -0.035509999999999944"/>
-    <mass value="0.0043107049436968805"/>
-    <inertia ixx="0.0" ixy="0.0" ixz="0.0" iyy="0.0" iyz="0.0" izz="0.0"/>
-  </inertial>
-  <visual>
-    <origin rpy="0 0 0" xyz="0.024889 -0.106281 -0.03591"/>
-    <geometry>
-      <mesh filename="package://ppp_description/meshes/axis_1.stl" scale="0.001 0.001 0.001"/>
-    </geometry>
-    <material name="silver"/>
-  </visual>
-  <collision>
-    <origin rpy="0 0 0" xyz="0.024889 -0.106281 -0.03591"/>
-    <geometry>
-      <mesh filename="package://ppp_description/meshes/axis_1.stl" scale="0.001 0.001 0.001"/>
-    </geometry>
-  </collision>
-</link>
-<link name="holder_1">
-  <inertial>
-    <origin rpy="0 0 0" xyz="0.0011550098836461376 -3.867842181329295e-06 -0.0024145150891157104"/>
-    <mass value="0.006489971019909515"/>
-    <inertia ixx="1e-06" ixy="-0.0" ixz="0.0" iyy="0.0" iyz="-0.0" izz="1e-06"/>
-  </inertial>
-  <visual>
-    <origin rpy="0 0 0" xyz="-0.00015 -0.106281 -0.0145"/>
-    <geometry>
-      <mesh filename="package://ppp_description/meshes/holder_1.stl" scale="0.001 0.001 0.001"/>
-    </geometry>
-    <material name="silver"/>
-  </visual>
-  <collision>
-    <origin rpy="0 0 0" xyz="-0.00015 -0.106281 -0.0145"/>
-    <geometry>
-      <mesh filename="package://ppp_description/meshes/holder_1.stl" scale="0.001 0.001 0.001"/>
-    </geometry>
-  </collision>
-</link>
-<link name="axis_main_1">
-  <inertial>
-    <origin rpy="0 0 0" xyz="4.181978385548596e-13 -1.1035397275149794e-07 -0.003749999999999993"/>
-    <mass value="0.003193114773108801"/>
-    <inertia ixx="0.0" ixy="-0.0" ixz="-0.0" iyy="0.0" iyz="-0.0" izz="0.0"/>
-  </inertial>
-  <visual>
-    <origin rpy="0 0 0" xyz="-0.00015 -0.106281 -0.022"/>
-    <geometry>
-      <mesh filename="package://ppp_description/meshes/axis_main_1.stl" scale="0.001 0.001 0.001"/>
-    </geometry>
-    <material name="silver"/>
-  </visual>
-  <collision>
-    <origin rpy="0 0 0" xyz="-0.00015 -0.106281 -0.022"/>
-    <geometry>
-      <mesh filename="package://ppp_description/meshes/axis_main_1.stl" scale="0.001 0.001 0.001"/>
-    </geometry>
-  </collision>
-</link>
-<!--FORWARD_WHEEL-->
 <link name="IMU_1">
   <inertial>
@@ -525,4 +443,9 @@
   <child link="12GAN20__1__Mirror__1"/>
 </joint>
+<joint name="Rigid19" type="fixed">
+  <origin rpy="0 0 0" xyz="-0.120925 -0.014338 0.022"/>
+  <parent link="base_link"/>
+  <child link="Forward_wheel_1"/>
+</joint>
 <joint name="Rigid21" type="fixed">
   <origin rpy="0 0 0" xyz="-0.163494 -0.014338 0.11"/>
@@ -530,5 +453,5 @@
   <child link="forward_top_1_1"/>
 </joint>
-<joint name="base_to_forward_top" type="fixed">
+<joint name="Rigid22" type="fixed">
   <origin rpy="0 0 0" xyz="0.004866 -0.157868 0.11"/>
   <parent link="base_link"/>
@@ -555,34 +478,3 @@
   <child link="IMU_1"/>
 </joint>
-<!--FORWARD_WHEEL-->
-<joint name="Rigid22" type="fixed">
-  <origin rpy="0 0 0" xyz="-0.014 0.117931 0.022"/>
-  <parent link="base_link"/>
-  <child link="FW_baise_1"/>
-</joint>
-<joint name="Rev26" type="continuous">
-  <origin rpy="0 0 0" xyz="0.033039 0.0 -0.03551"/>
-  <parent link="axis_1"/>
-  <child link="wheel__1__1"/>
-  <axis xyz="-0.0 -1.0 -0.0"/>
-</joint>
-<joint name="Rev27" type="continuous">
-  <origin rpy="0 0 0" xyz="-0.025039 0.0 0.02141"/>
-  <parent link="holder_1"/>
-  <child link="axis_1"/>
-  <axis xyz="0.0 1.0 0.0"/>
-</joint>
-<joint name="Rev28" type="continuous">
-  <origin rpy="0 0 0" xyz="0.0 0.0 -0.0075"/>
-  <parent link="axis_main_1"/>
-  <child link="holder_1"/>
-  <axis xyz="-0.0 0.0 -1.0"/>
-</joint>
-<joint name="Rev29" type="continuous">
-  <origin rpy="0 0 0" xyz="0.01415 -0.01165 0.0"/>
-  <parent link="FW_baise_1"/>
-  <child link="axis_main_1"/>
-  <axis xyz="0.0 -0.0 -1.0"/>
-</joint>
-<!--FORWARD_WHEEL-->
 </robot>

Commit message: fix odom

File: src/ppp90_description/urdf/ppp90.xacro (robot description, xacro)
@@ -364,5 +364,5 @@
   </collision>
 </link>
-<link name="IMU_1">
+<link name="base_imu_link">
   <inertial>
     <origin rpy="0 0 0" xyz="-4.3047029232856637e-07 -9.471075246465788e-08 0.007500000000000041"/>
@@ -476,5 +476,5 @@
   <origin rpy="0 0 0" xyz="-0.159074 -0.014338 0.033"/>
   <parent link="base_link"/>
-  <child link="IMU_1"/>
+  <child link="base_imu_link"/>
 </joint>
 </robot>

File: src/ppp_description/urdf/ppp.xacro (robot description, xacro)
@@ -349,5 +349,5 @@
 </link>
 <!--FORWARD_WHEEL-->
-<link name="IMU_1">
+<link name="base_imu_link">
   <inertial>
     <origin rpy="0 0 0" xyz="2.3440450969136606e-16 4.815371235089572e-07 0.008500000000000056"/>
@@ -563,5 +563,5 @@
   <origin rpy="0 0 0" xyz="-0.001 0.14314 0.033"/>
   <parent link="base_link"/>
-  <child link="IMU_1"/>
+  <child link="base_imu_link"/>
 </joint>
 <joint name="Rigid21" type="fixed">

Commit message: add some conf

File: src/ppp90_description/urdf/ppp90.xacro (robot description, xacro)
@@ -73,14 +73,15 @@
     <origin rpy="0 0 0" xyz="0.027494 -0.13623 -0.08983"/>
     <geometry>
+      <box size="0.001 0.0005 0.00035"/>
+      <!-- <mesh filename="package://ppp90_description/meshes/sonyc_1.stl" scale="0.001 0.001 0.001"/> -->
+    </geometry>
+    <material name="silver"/>
+  </visual>
+  <!-- <collision>
+    <origin rpy="0 0 0" xyz="0.027494 -0.13623 -0.08983"/>
+    <geometry>
       <mesh filename="package://ppp90_description/meshes/sonyc_1.stl" scale="0.001 0.001 0.001"/>
     </geometry>
-    <material name="silver"/>
-  </visual>
-  <collision>
-    <origin rpy="0 0 0" xyz="0.027494 -0.13623 -0.08983"/>
-    <geometry>
-      <mesh filename="package://ppp90_description/meshes/sonyc_1.stl" scale="0.001 0.001 0.001"/>
-    </geometry>
-  </collision>
+  </collision> -->
 </link>
 <link name="sonyc_Mirror__1">
@@ -93,14 +94,15 @@
     <origin rpy="0 0 0" xyz="0.001494 0.164906 -0.08983"/>
     <geometry>
+      <box size="0.001 0.0005 0.00035"/>
+      <!-- <mesh filename="package://ppp90_description/meshes/sonyc_Mirror__1.stl" scale="0.001 0.001 0.001"/> -->
+    </geometry>
+    <material name="silver"/>
+  </visual>
+  <!-- <collision>
+    <origin rpy="0 0 0" xyz="0.001494 0.164906 -0.08983"/>
+    <geometry>
       <mesh filename="package://ppp90_description/meshes/sonyc_Mirror__1.stl" scale="0.001 0.001 0.001"/>
     </geometry>
-    <material name="silver"/>
-  </visual>
-  <collision>
-    <origin rpy="0 0 0" xyz="0.001494 0.164906 -0.08983"/>
-    <geometry>
-      <mesh filename="package://ppp90_description/meshes/sonyc_Mirror__1.stl" scale="0.001 0.001 0.001"/>
-    </geometry>
-  </collision>
+  </collision> -->
 </link>
 <link name="sonyc__1__1">
@@ -113,14 +115,15 @@
     <origin rpy="0 0 0" xyz="0.169414 0.001361 -0.06983"/>
     <geometry>
+      <box size="0.001 0.0005 0.00035"/>
+      <!-- <mesh filename="package://ppp90_description/meshes/sonyc__1__1.stl" scale="0.001 0.001 0.001"/> -->
+    </geometry>
+    <material name="silver"/>
+  </visual>
+  <!-- <collision>
+    <origin rpy="0 0 0" xyz="0.169414 0.001361 -0.06983"/>
+    <geometry>
       <mesh filename="package://ppp90_description/meshes/sonyc__1__1.stl" scale="0.001 0.001 0.001"/>
     </geometry>
-    <material name="silver"/>
-  </visual>
-  <collision>
-    <origin rpy="0 0 0" xyz="0.169414 0.001361 -0.06983"/>
-    <geometry>
-      <mesh filename="package://ppp90_description/meshes/sonyc__1__1.stl" scale="0.001 0.001 0.001"/>
-    </geometry>
-  </collision>
+  </collision> -->
 </link>
 <link name="nema17_1">
@@ -397,15 +400,15 @@
 </joint>
 <joint name="Rigid5" type="fixed">
-  <origin rpy="0 0 0" xyz="-0.027494 0.13623 0.08983"/>
+  <origin rpy="0 0 1.5" xyz="-0.027494 0.13623 0.08983"/>
   <parent link="base_link"/>
   <child link="sonyc_1"/>
 </joint>
 <joint name="Rigid6" type="fixed">
-  <origin rpy="0 0 0" xyz="-0.001494 -0.164906 0.08983"/>
+  <origin rpy="0 0 -1.65" xyz="-0.001494 -0.164906 0.08983"/>
   <parent link="base_link"/>
   <child link="sonyc_Mirror__1"/>
 </joint>
 <joint name="Rigid7" type="fixed">
-  <origin rpy="0 0 0" xyz="-0.169414 -0.001361 0.06983"/>
+  <origin rpy="0 0 -3.14159" xyz="-0.169414 -0.001361 0.06983"/>
   <parent link="base_link"/>
   <child link="sonyc__1__1"/>

Commit message: add localization config

File: src/ppp90_description/urdf/ppp90.xacro (robot description, xacro)
@@ -400,5 +400,5 @@
 </joint>
 <joint name="Rigid5" type="fixed">
-  <origin rpy="0 0 1.5" xyz="-0.027494 0.13623 0.08983"/>
+  <origin rpy="0 0 1.50" xyz="-0.027494 0.13623 0.08983"/>
   <parent link="base_link"/>
   <child link="sonyc_1"/>
