Commit message: fix v1 acml

File: src/ppp90_description/urdf/ppp90.xacro (robot description, xacro)
@@ -6,10 +6,10 @@
 <link name="base_link">
   <inertial>
-    <origin rpy="0 0 3.14159" xyz="-0.006384053079489355 -0.014519040269770902 0.03416379967065736"/>
+    <origin rpy="0 0 0" xyz="-0.006384053079489355 -0.014519040269770902 0.03416379967065736"/>
     <mass value="5.029311101542255"/>
     <inertia ixx="0.037081" ixy="0.000111" ixz="-0.001835" iyy="0.04462" iyz="2e-05" izz="0.070617"/>
   </inertial>
   <visual>
-    <origin rpy="0 0 3.14159" xyz="0 0 0"/>
+    <origin rpy="0 0 0" xyz="0 0 0"/>
     <geometry>
       <mesh filename="package://ppp90_description/meshes/base_link.stl" scale="0.001 0.001 0.001"/>
@@ -18,5 +18,5 @@
   </visual>
   <collision>
-    <origin rpy="0 0 3.14159" xyz="0 0 0"/>
+    <origin rpy="0 0 0" xyz="0 0 0"/>
     <geometry>
       <mesh filename="package://ppp90_description/meshes/base_link.stl" scale="0.001 0.001 0.001"/>
@@ -26,10 +26,10 @@
 <link name="wheel_1">
   <inertial>
-    <origin rpy="0 0 3.14159" xyz="-6.348907630078851e-05 -0.01199981164843078 -0.00029175072703385013"/>
+    <origin rpy="0 0 0" xyz="-6.348907630078851e-05 -0.01199981164843078 -0.00029175072703385013"/>
     <mass value="0.7647072407364309"/>
     <inertia ixx="0.000285" ixy="-0.0" ixz="0.0" iyy="0.000502" iyz="0.0" izz="0.000285"/>
   </inertial>
   <visual>
-    <origin rpy="0 0 3.14159" xyz="0.014494 -0.129921 -0.024125"/>
+    <origin rpy="0 0 0" xyz="0.014494 -0.129921 -0.024125"/>
     <geometry>
       <mesh filename="package://ppp90_description/meshes/wheel_1.stl" scale="0.001 0.001 0.001"/>
@@ -38,5 +38,5 @@
   </visual>
   <collision>
-    <origin rpy="0 0 3.14159" xyz="0.014494 -0.129921 -0.024125"/>
+    <origin rpy="0 0 0" xyz="0.014494 -0.129921 -0.024125"/>
     <geometry>
       <mesh filename="package://ppp90_description/meshes/wheel_1.stl" scale="0.001 0.001 0.001"/>
@@ -46,10 +46,10 @@
 <link name="wheel_Mirror__1">
   <inertial>
-    <origin rpy="0 0 3.14159" xyz="0.0001513902914462642 -0.011999864080914024 0.00026807201904406955"/>
+    <origin rpy="0 0 0" xyz="0.0001513902914462642 -0.011999864080914024 0.00026807201904406955"/>
     <mass value="0.7647072407364308"/>
     <inertia ixx="0.000285" ixy="-0.0" ixz="0.0" iyy="0.000502" iyz="0.0" izz="0.000285"/>
   </inertial>
   <visual>
-    <origin rpy="0 0 3.14159" xyz="0.014491 0.136188 -0.024125"/>
+    <origin rpy="0 0 0" xyz="0.014491 0.136188 -0.024125"/>
     <geometry>
       <mesh filename="package://ppp90_description/meshes/wheel_Mirror__1.stl" scale="0.001 0.001 0.001"/>
@@ -58,5 +58,5 @@
   </visual>
   <collision>
-    <origin rpy="0 0 3.14159" xyz="0.014491 0.136188 -0.024125"/>
+    <origin rpy="0 0 0" xyz="0.014491 0.136188 -0.024125"/>
     <geometry>
       <mesh filename="package://ppp90_description/meshes/wheel_Mirror__1.stl" scale="0.001 0.001 0.001"/>
@@ -66,10 +66,10 @@
 <link name="sonyc_1">
   <inertial>
-    <origin rpy="0 0 3.14159" xyz="0.013000365548618742 -0.010235515019977243 5.0631813087009814e-05"/>
+    <origin rpy="0 0 0" xyz="0.013000365548618742 -0.010235515019977243 5.0631813087009814e-05"/>
     <mass value="0.0252883585593009"/>
     <inertia ixx="1e-06" ixy="0.0" ixz="0.0" iyy="5e-06" iyz="-0.0" izz="5e-06"/>
   </inertial>
   <visual>
-    <origin rpy="0 0 3.14159" xyz="0.027494 -0.13623 -0.08983"/>
+    <origin rpy="0 0 0" xyz="0.027494 -0.13623 -0.08983"/>
     <geometry>
       <box size="0.001 0.0005 0.00035"/>
@@ -79,5 +79,5 @@
   </visual>
   <!-- <collision>
-    <origin rpy="0 0 3.14159" xyz="0.027494 -0.13623 -0.08983"/>
+    <origin rpy="0 0 0" xyz="0.027494 -0.13623 -0.08983"/>
     <geometry>
       <mesh filename="package://ppp90_description/meshes/sonyc_1.stl" scale="0.001 0.001 0.001"/>
@@ -87,10 +87,10 @@
 <link name="sonyc_Mirror__1">
   <inertial>
-    <origin rpy="0 0 3.14159" xyz="-0.012999634451381028 0.010235325598471623 5.063181308698206e-05"/>
+    <origin rpy="0 0 0" xyz="-0.012999634451381028 0.010235325598471623 5.063181308698206e-05"/>
     <mass value="0.025288358559300887"/>
     <inertia ixx="1e-06" ixy="-0.0" ixz="0.0" iyy="5e-06" iyz="0.0" izz="5e-06"/>
   </inertial>
   <visual>
-    <origin rpy="0 0 3.14159" xyz="0.001494 0.164906 -0.08983"/>
+    <origin rpy="0 0 0" xyz="0.001494 0.164906 -0.08983"/>
     <geometry>
       <box size="0.001 0.0005 0.00035"/>
@@ -100,5 +100,5 @@
   </visual>
   <!-- <collision>
-    <origin rpy="0 0 3.14159" xyz="0.001494 0.164906 -0.08983"/>
+    <origin rpy="0 0 0" xyz="0.001494 0.164906 -0.08983"/>
     <geometry>
       <mesh filename="package://ppp90_description/meshes/sonyc_Mirror__1.stl" scale="0.001 0.001 0.001"/>
@@ -108,10 +108,10 @@
 <link name="sonyc__1__1">
   <inertial>
-    <origin rpy="0 0 3.14159" xyz="0.010235448068739439 -0.013000419106913505 5.063181308698206e-05"/>
+    <origin rpy="0 0 0" xyz="0.010235448068739439 -0.013000419106913505 5.063181308698206e-05"/>
     <mass value="0.0252883585593009"/>
     <inertia ixx="5e-06" ixy="-0.0" ixz="0.0" iyy="1e-06" iyz="0.0" izz="5e-06"/>
   </inertial>
   <visual>
-    <origin rpy="0 0 3.14159" xyz="0.169414 0.001361 -0.06983"/>
+    <origin rpy="0 0 0" xyz="0.169414 0.001361 -0.06983"/>
     <geometry>
       <box size="0.001 0.0005 0.00035"/>
@@ -121,5 +121,5 @@
   </visual>
   <!-- <collision>
-    <origin rpy="0 0 3.14159" xyz="0.169414 0.001361 -0.06983"/>
+    <origin rpy="0 0 0" xyz="0.169414 0.001361 -0.06983"/>
     <geometry>
       <mesh filename="package://ppp90_description/meshes/sonyc__1__1.stl" scale="0.001 0.001 0.001"/>
@@ -129,10 +129,10 @@
 <link name="nema17_1">
   <inertial>
-    <origin rpy="0 0 3.14159" xyz="-6.709208478471174e-07 -0.00334258185473002 0.02118013525930306"/>
+    <origin rpy="0 0 0" xyz="-6.709208478471174e-07 -0.00334258185473002 0.02118013525930306"/>
     <mass value="0.1838412954712099"/>
     <inertia ixx="5.2e-05" ixy="-0.0" ixz="-0.0" iyy="5.3e-05" iyz="0.0" izz="5.2e-05"/>
   </inertial>
   <visual>
-    <origin rpy="0 0 3.14159" xyz="0.014494 -0.084071 -0.003"/>
+    <origin rpy="0 0 0" xyz="0.014494 -0.084071 -0.003"/>
     <geometry>
       <mesh filename="package://ppp90_description/meshes/nema17_1.stl" scale="0.001 0.001 0.001"/>
@@ -141,5 +141,5 @@
   </visual>
   <collision>
-    <origin rpy="0 0 3.14159" xyz="0.014494 -0.084071 -0.003"/>
+    <origin rpy="0 0 0" xyz="0.014494 -0.084071 -0.003"/>
     <geometry>
       <mesh filename="package://ppp90_description/meshes/nema17_1.stl" scale="0.001 0.001 0.001"/>
@@ -149,10 +149,10 @@
 <link name="nema17_Mirror__1">
   <inertial>
-    <origin rpy="0 0 3.14159" xyz="-5.975012162888829e-06 0.00334264208445903 0.02118013525930306"/>
+    <origin rpy="0 0 0" xyz="-5.975012162888829e-06 0.00334264208445903 0.02118013525930306"/>
     <mass value="0.1838412954712099"/>
     <inertia ixx="5.2e-05" ixy="-0.0" ixz="-0.0" iyy="5.3e-05" iyz="-0.0" izz="5.2e-05"/>
   </inertial>
   <visual>
-    <origin rpy="0 0 3.14159" xyz="0.014528 0.113338 -0.003"/>
+    <origin rpy="0 0 0" xyz="0.014528 0.113338 -0.003"/>
     <geometry>
       <mesh filename="package://ppp90_description/meshes/nema17_Mirror__1.stl" scale="0.001 0.001 0.001"/>
@@ -161,5 +161,5 @@
   </visual>
   <collision>
-    <origin rpy="0 0 3.14159" xyz="0.014528 0.113338 -0.003"/>
+    <origin rpy="0 0 0" xyz="0.014528 0.113338 -0.003"/>
     <geometry>
       <mesh filename="package://ppp90_description/meshes/nema17_Mirror__1.stl" scale="0.001 0.001 0.001"/>
@@ -169,10 +169,10 @@
 <link name="12GAN20__1__1">
   <inertial>
-    <origin rpy="0 0 3.14159" xyz="3.268980405812805e-08 -3.387342204674848e-06 0.011857871337072723"/>
+    <origin rpy="0 0 0" xyz="3.268980405812805e-08 -3.387342204674848e-06 0.011857871337072723"/>
     <mass value="0.023492103087793172"/>
     <inertia ixx="1e-06" ixy="-0.0" ixz="-0.0" iyy="2e-06" iyz="-0.0" izz="0.0"/>
   </inertial>
   <visual>
-    <origin rpy="0 0 3.14159" xyz="0.096453 0.12774 -0.001"/>
+    <origin rpy="0 0 0" xyz="0.096453 0.12774 -0.001"/>
     <geometry>
       <mesh filename="package://ppp90_description/meshes/12GAN20__1__1.stl" scale="0.001 0.001 0.001"/>
@@ -181,5 +181,5 @@
   </visual>
   <collision>
-    <origin rpy="0 0 3.14159" xyz="0.096453 0.12774 -0.001"/>
+    <origin rpy="0 0 0" xyz="0.096453 0.12774 -0.001"/>
     <geometry>
       <mesh filename="package://ppp90_description/meshes/12GAN20__1__1.stl" scale="0.001 0.001 0.001"/>
@@ -189,10 +189,10 @@
 <link name="brush_1">
   <inertial>
-    <origin rpy="0 0 3.14159" xyz="-6.629561645765669e-07 -8.680417363238213e-07 -0.0022204199308318013"/>
+    <origin rpy="0 0 0" xyz="-6.629561645765669e-07 -8.680417363238213e-07 -0.0022204199308318013"/>
     <mass value="0.014937067448072668"/>
     <inertia ixx="1e-06" ixy="0.0" ixz="0.0" iyy="1e-06" iyz="0.0" izz="2e-06"/>
   </inertial>
   <visual>
-    <origin rpy="0 0 3.14159" xyz="0.096455 0.12775 0.001"/>
+    <origin rpy="0 0 0" xyz="0.096455 0.12775 0.001"/>
     <geometry>
       <mesh filename="package://ppp90_description/meshes/brush_1.stl" scale="0.001 0.001 0.001"/>
@@ -201,5 +201,5 @@
   </visual>
   <collision>
-    <origin rpy="0 0 3.14159" xyz="0.096455 0.12775 0.001"/>
+    <origin rpy="0 0 0" xyz="0.096455 0.12775 0.001"/>
     <geometry>
       <mesh filename="package://ppp90_description/meshes/brush_1.stl" scale="0.001 0.001 0.001"/>
@@ -209,10 +209,10 @@
 <link name="brush_Mirror__1">
   <inertial>
-    <origin rpy="0 0 3.14159" xyz="5.998655124295205e-07 3.438472244571278e-07 -0.0022204199308317827"/>
+    <origin rpy="0 0 0" xyz="5.998655124295205e-07 3.438472244571278e-07 -0.0022204199308317827"/>
     <mass value="0.014937067448072664"/>
     <inertia ixx="1e-06" ixy="0.0" ixz="-0.0" iyy="1e-06" iyz="0.0" izz="2e-06"/>
   </inertial>
   <visual>
-    <origin rpy="0 0 3.14159" xyz="0.096451 -0.099054 0.001"/>
+    <origin rpy="0 0 0" xyz="0.096451 -0.099054 0.001"/>
     <geometry>
       <mesh filename="package://ppp90_description/meshes/brush_Mirror__1.stl" scale="0.001 0.001 0.001"/>
@@ -221,5 +221,5 @@
   </visual>
   <collision>
-    <origin rpy="0 0 3.14159" xyz="0.096451 -0.099054 0.001"/>
+    <origin rpy="0 0 0" xyz="0.096451 -0.099054 0.001"/>
     <geometry>
       <mesh filename="package://ppp90_description/meshes/brush_Mirror__1.stl" scale="0.001 0.001 0.001"/>
@@ -229,10 +229,10 @@
 <link name="12GAN20__1__Mirror__1">
   <inertial>
-    <origin rpy="0 0 3.14159" xyz="2.061205277625877e-06 -6.450130101642859e-06 0.011857871337072723"/>
+    <origin rpy="0 0 0" xyz="2.061205277625877e-06 -6.450130101642859e-06 0.011857871337072723"/>
     <mass value="0.02349210308779317"/>
     <inertia ixx="1e-06" ixy="0.0" ixz="-0.0" iyy="2e-06" iyz="0.0" izz="0.0"/>
   </inertial>
   <visual>
-    <origin rpy="0 0 3.14159" xyz="0.096451 -0.099054 -0.001"/>
+    <origin rpy="0 0 0" xyz="0.096451 -0.099054 -0.001"/>
     <geometry>
       <mesh filename="package://ppp90_description/meshes/12GAN20__1__Mirror__1.stl" scale="0.001 0.001 0.001"/>
@@ -241,5 +241,5 @@
   </visual>
   <collision>
-    <origin rpy="0 0 3.14159" xyz="0.096451 -0.099054 -0.001"/>
+    <origin rpy="0 0 0" xyz="0.096451 -0.099054 -0.001"/>
     <geometry>
       <mesh filename="package://ppp90_description/meshes/12GAN20__1__Mirror__1.stl" scale="0.001 0.001 0.001"/>
@@ -249,10 +249,10 @@
 <link name="Forward_wheel_1">
   <inertial>
-    <origin rpy="0 0 3.14159" xyz="4.803445236845061e-07 -9.471071670506814e-08 -0.001437450709413722"/>
+    <origin rpy="0 0 0" xyz="4.803445236845061e-07 -9.471071670506814e-08 -0.001437450709413722"/>
     <mass value="0.0061871055650105375"/>
     <inertia ixx="0.0" ixy="0.0" ixz="0.0" iyy="0.0" iyz="0.0" izz="1e-06"/>
   </inertial>
   <visual>
-    <origin rpy="0 0 3.14159" xyz="0.120925 0.014338 -0.022"/>
+    <origin rpy="0 0 0" xyz="0.120925 0.014338 -0.022"/>
     <geometry>
       <mesh filename="package://ppp90_description/meshes/Forward_wheel_1.stl" scale="0.001 0.001 0.001"/>
@@ -261,5 +261,5 @@
   </visual>
   <collision>
-    <origin rpy="0 0 3.14159" xyz="0.120925 0.014338 -0.022"/>
+    <origin rpy="0 0 0" xyz="0.120925 0.014338 -0.022"/>
     <geometry>
       <mesh filename="package://ppp90_description/meshes/Forward_wheel_1.stl" scale="0.001 0.001 0.001"/>
@@ -269,10 +269,10 @@
 <link name="forward_top_1_1">
   <inertial>
-    <origin rpy="0 0 3.14159" xyz="0.09472417565339834 0.0650218967379826 0.0004895173930853647"/>
+    <origin rpy="0 0 0" xyz="0.09472417565339834 0.0650218967379826 0.0004895173930853647"/>
     <mass value="0.48710215659029577"/>
     <inertia ixx="0.000784" ixy="-0.000235" ixz="1e-06" iyy="0.00099" iyz="1e-06" izz="0.001773"/>
   </inertial>
   <visual>
-    <origin rpy="0 0 3.14159" xyz="0.163494 0.014338 -0.11"/>
+    <origin rpy="0 0 0" xyz="0.163494 0.014338 -0.11"/>
     <geometry>
       <mesh filename="package://ppp90_description/meshes/forward_top_1_1.stl" scale="0.001 0.001 0.001"/>
@@ -281,5 +281,5 @@
   </visual>
   <collision>
-    <origin rpy="0 0 3.14159" xyz="0.163494 0.014338 -0.11"/>
+    <origin rpy="0 0 0" xyz="0.163494 0.014338 -0.11"/>
     <geometry>
       <mesh filename="package://ppp90_description/meshes/forward_top_1_1.stl" scale="0.001 0.001 0.001"/>
@@ -289,10 +289,10 @@
 <link name="forward_top_1_Mirror__1">
   <inertial>
-    <origin rpy="0 0 3.14159" xyz="-0.07359144458337072 0.07845770313065512 0.0004895171912022017"/>
+    <origin rpy="0 0 0" xyz="-0.07359144458337072 0.07845770313065512 0.0004895171912022017"/>
     <mass value="0.48710223650351714"/>
     <inertia ixx="0.000784" ixy="0.000234" ixz="1e-06" iyy="0.00099" iyz="-1e-06" izz="0.001773"/>
   </inertial>
   <visual>
-    <origin rpy="0 0 3.14159" xyz="-0.004866 0.157868 -0.11"/>
+    <origin rpy="0 0 0" xyz="-0.004866 0.157868 -0.11"/>
     <geometry>
       <mesh filename="package://ppp90_description/meshes/forward_top_1_Mirror__1.stl" scale="0.001 0.001 0.001"/>
@@ -301,5 +301,5 @@
   </visual>
   <collision>
-    <origin rpy="0 0 3.14159" xyz="-0.004866 0.157868 -0.11"/>
+    <origin rpy="0 0 0" xyz="-0.004866 0.157868 -0.11"/>
     <geometry>
       <mesh filename="package://ppp90_description/meshes/forward_top_1_Mirror__1.stl" scale="0.001 0.001 0.001"/>
@@ -309,10 +309,10 @@
 <link name="back_top_1">
   <inertial>
-    <origin rpy="0 0 3.14159" xyz="0.06983870948069765 0.07365312062764642 -0.001088719949768488"/>
+    <origin rpy="0 0 0" xyz="0.06983870948069765 0.07365312062764642 -0.001088719949768488"/>
     <mass value="0.23560428740017997"/>
     <inertia ixx="0.000537" ixy="-0.000345" ixz="1.3e-05" iyy="0.00038" iyz="1.8e-05" izz="0.000907"/>
   </inertial>
   <visual>
-    <origin rpy="0 0 3.14159" xyz="-0.004866 0.157868 -0.11"/>
+    <origin rpy="0 0 0" xyz="-0.004866 0.157868 -0.11"/>
     <geometry>
       <mesh filename="package://ppp90_description/meshes/back_top_1.stl" scale="0.001 0.001 0.001"/>
@@ -321,5 +321,5 @@
   </visual>
   <collision>
-    <origin rpy="0 0 3.14159" xyz="-0.004866 0.157868 -0.11"/>
+    <origin rpy="0 0 0" xyz="-0.004866 0.157868 -0.11"/>
     <geometry>
       <mesh filename="package://ppp90_description/meshes/back_top_1.stl" scale="0.001 0.001 0.001"/>
@@ -329,10 +329,10 @@
 <link name="back_top2_1">
   <inertial>
-    <origin rpy="0 0 3.14159" xyz="0.05870883159733394 -0.05499680190680151 0.0004968868769273244"/>
+    <origin rpy="0 0 0" xyz="0.05870883159733394 -0.05499680190680151 0.0004968868769273244"/>
     <mass value="0.18961170684744505"/>
     <inertia ixx="0.000183" ixy="0.000153" ixz="-1e-06" iyy="0.000249" iyz="1e-06" izz="0.000432"/>
   </inertial>
   <visual>
-    <origin rpy="0 0 3.14159" xyz="-0.004866 -0.129192 -0.11"/>
+    <origin rpy="0 0 0" xyz="-0.004866 -0.129192 -0.11"/>
     <geometry>
       <mesh filename="package://ppp90_description/meshes/back_top2_1.stl" scale="0.001 0.001 0.001"/>
@@ -341,5 +341,5 @@
   </visual>
   <collision>
-    <origin rpy="0 0 3.14159" xyz="-0.004866 -0.129192 -0.11"/>
+    <origin rpy="0 0 0" xyz="-0.004866 -0.129192 -0.11"/>
     <geometry>
       <mesh filename="package://ppp90_description/meshes/back_top2_1.stl" scale="0.001 0.001 0.001"/>
@@ -349,10 +349,10 @@
 <link name="Lidar_1">
   <inertial>
-    <origin rpy="0 0 3.14159" xyz="1.561464430532844e-07 1.323739005389124e-08 0.03500000000000007"/>
+    <origin rpy="0 0 0" xyz="1.561464430532844e-07 1.323739005389124e-08 0.03500000000000007"/>
     <mass value="2.114723824855799"/>
     <inertia ixx="0.001511" ixy="-0.0" ixz="0.0" iyy="0.001511" iyz="-0.0" izz="0.001295"/>
   </inertial>
   <visual>
-    <origin rpy="0 0 3.14159" xyz="0.110814 0.014417 -0.112"/>
+    <origin rpy="0 0 0" xyz="0.110814 0.014417 -0.112"/>
     <geometry>
       <mesh filename="package://ppp90_description/meshes/Lidar_1.stl" scale="0.001 0.001 0.001"/>
@@ -361,5 +361,5 @@
   </visual>
   <collision>
-    <origin rpy="0 0 3.14159" xyz="0.110814 0.014417 -0.112"/>
+    <origin rpy="0 0 0" xyz="0.110814 0.014417 -0.112"/>
     <geometry>
       <mesh filename="package://ppp90_description/meshes/Lidar_1.stl" scale="0.001 0.001 0.001"/>
@@ -369,10 +369,10 @@
 <link name="base_imu_link">
   <inertial>
-    <origin rpy="0 0 3.14159" xyz="-4.3047029232856637e-07 -9.471075246465788e-08 0.007500000000000041"/>
+    <origin rpy="0 0 0" xyz="-4.3047029232856637e-07 -9.471075246465788e-08 0.007500000000000041"/>
     <mass value="0.011774999999999999"/>
     <inertia ixx="1e-06" ixy="0.0" ixz="0.0" iyy="0.0" iyz="-0.0" izz="0.0"/>
   </inertial>
   <visual>
-    <origin rpy="0 0 3.14159" xyz="0.159074 0.014338 -0.033"/>
+    <origin rpy="0 0 0" xyz="0.159074 0.014338 -0.033"/>
     <geometry>
       <mesh filename="package://ppp90_description/meshes/IMU_1.stl" scale="0.001 0.001 0.001"/>
@@ -381,5 +381,5 @@
   </visual>
   <collision>
-    <origin rpy="0 0 3.14159" xyz="0.159074 0.014338 -0.033"/>
+    <origin rpy="0 0 0" xyz="0.159074 0.014338 -0.033"/>
     <geometry>
       <mesh filename="package://ppp90_description/meshes/IMU_1.stl" scale="0.001 0.001 0.001"/>

Commit message: change move base

File: src/ppp90_description/urdf/ppp90.xacro (robot description, xacro)
@@ -4,4 +4,10 @@
 <xacro:include filename="$(find ppp90_description)/urdf/ppp90.trans" />
 <xacro:include filename="$(find ppp90_description)/urdf/ppp90.gazebo" />
+<link name="base_footprint"/>
+<joint name="base_joint" type="fixed">
+    <parent link="base_footprint"/>
+    <child link="base_link"/>
+    <origin xyz="0.0 0.0 0.010" rpy="0 0 0"/>
+</joint>
 <link name="base_link">
   <inertial>

Commit message: fix emulation & controllers

File: src/ppp90_description/urdf/ppp90.xacro (robot description, xacro)
@@ -5,9 +5,4 @@
 <xacro:include filename="$(find ppp90_description)/urdf/ppp90.gazebo" />
 <link name="base_link">
-  <inertial>
-    <origin rpy="0 0 0" xyz="-0.006384053079489355 -0.014519040269770902 0.03416379967065736"/>
-    <mass value="5.029311101542255"/>
-    <inertia ixx="0.037081" ixy="0.000111" ixz="-0.001835" iyy="0.04462" iyz="2e-05" izz="0.070617"/>
-  </inertial>
   <visual>
     <origin rpy="0 0 0" xyz="0 0 0"/>

Commit message: v2

File: src/ppp90_description/urdf/ppp90.xacro (robot description, xacro)
@@ -250,5 +250,5 @@
   </inertial>
   <visual>
-    <origin rpy="0 0 0" xyz="-0.0052579363728012885 -0.10377441452254206 -0.01"/>
+    <origin rpy="0 0 0" xyz="0.0052579363728012885 0.10377441452254206 0.014658078584554117"/>
     <geometry>
       <mesh filename="package://ppp90_description/meshes/Forward_wheel.stl" scale="0.001 0.001 0.001"/>
@@ -257,5 +257,5 @@
   </visual>
   <collision>
-    <origin rpy="0 0 0" xyz="0 0 0"/>
+    <origin rpy="0 0 0" xyz="0.0052579363728012885 0.10377441452254206 0.014658078584554117"/>
     <geometry>
       <mesh filename="package://ppp90_description/meshes/Forward_wheel.stl" scale="0.001 0.001 0.001"/>
@@ -344,5 +344,5 @@
 </link>
 <joint name="Rigid19" type="fixed">
-  <origin rpy="0 0 0" xyz="-0.120925 -0.014338 0.022"/>
+  <origin rpy="0 0 1.5708" xyz="-0.120925 -0.014338 0.022"/>
   <parent link="base_link"/>
   <child link="Forward_wheel"/>

Commit message: v3

File: src/ppp90_description/urdf/ppp90.xacro (robot description, xacro)
@@ -245,10 +245,10 @@
 <link name="Forward_wheel">
    <inertial>
-    <origin rpy="0 0 0" xyz="0.0052579363728012885 0.10377441452254206 0.014658078584554117"/>
+    <origin rpy="0 0 0" xyz="-0.0052579363728012885 -0.10377441452254206 -0.015"/>
     <mass value="0.0061871055650105375"/>
     <inertia ixx="0.0" ixy="-0.0" ixz="0.0" iyy="0.0" iyz="-0.0" izz="1e-06"/>
   </inertial>
   <visual>
-    <origin rpy="0 0 0" xyz="0.0052579363728012885 0.10377441452254206 0.014658078584554117"/>
+    <origin rpy="0 0 0" xyz="-0.0052579363728012885 -0.10377441452254206 -0.015"/>
     <geometry>
       <mesh filename="package://ppp90_description/meshes/Forward_wheel.stl" scale="0.001 0.001 0.001"/>
@@ -257,5 +257,5 @@
   </visual>
   <collision>
-    <origin rpy="0 0 0" xyz="0.0052579363728012885 0.10377441452254206 0.014658078584554117"/>
+    <origin rpy="0 0 0" xyz="-0.0052579363728012885 -0.10377441452254206 -0.015"/>
     <geometry>
       <mesh filename="package://ppp90_description/meshes/Forward_wheel.stl" scale="0.001 0.001 0.001"/>
