Commit message: turn model

File: src/ppp90_description/urdf/ppp90.xacro (robot description, xacro)
@@ -11,4 +11,9 @@
 </joint>
 <link name="base_link">
+  <inertial>
+    <origin rpy="0 0 0" xyz="0.006228517780792832 -0.014312684450430895 0.03416379967065732"/>
+    <mass value="5.029311101542255"/>
+    <inertia ixx="0.037081" ixy="0.000111" ixz="0.001835" iyy="0.04462" iyz="-2e-05" izz="0.070617"/>
+  </inertial>
   <visual>
     <origin rpy="0 0 0" xyz="0 0 0"/>
@@ -27,10 +32,10 @@
 <link name="wheel_1">
   <inertial>
-    <origin rpy="0 0 0" xyz="-6.348907630078851e-05 -0.01199981164843078 -0.00029175072703385013"/>
+    <origin rpy="0 0 0" xyz="6.395377760427118e-05 0.012000086928228931 -0.0002917507270338848"/>
     <mass value="0.7647072407364309"/>
-    <inertia ixx="0.000285" ixy="-0.0" ixz="0.0" iyy="0.000502" iyz="0.0" izz="0.000285"/>
-  </inertial>
-  <visual>
-    <origin rpy="0 0 0" xyz="0.014494 -0.129921 -0.024125"/>
+    <inertia ixx="0.000285" ixy="-0.0" ixz="-0.0" iyy="0.000502" iyz="-0.0" izz="0.000285"/>
+  </inertial>
+  <visual>
+    <origin rpy="0 0 0" xyz="-0.014338 0.158753 -0.024125"/>
     <geometry>
       <mesh filename="package://ppp90_description/meshes/wheel_1.stl" scale="0.001 0.001 0.001"/>
@@ -39,5 +44,5 @@
   </visual>
   <collision>
-    <origin rpy="0 0 0" xyz="0.014494 -0.129921 -0.024125"/>
+    <origin rpy="0 0 0" xyz="-0.014338 0.158753 -0.024125"/>
     <geometry>
       <mesh filename="package://ppp90_description/meshes/wheel_1.stl" scale="0.001 0.001 0.001"/>
@@ -47,10 +52,10 @@
 <link name="wheel_Mirror__1">
   <inertial>
-    <origin rpy="0 0 0" xyz="0.0001513902914462642 -0.011999864080914024 0.00026807201904406955"/>
+    <origin rpy="0 0 0" xyz="-0.00015092559014278847 0.01200013936071219 0.0002680720190440314"/>
     <mass value="0.7647072407364308"/>
-    <inertia ixx="0.000285" ixy="-0.0" ixz="0.0" iyy="0.000502" iyz="0.0" izz="0.000285"/>
-  </inertial>
-  <visual>
-    <origin rpy="0 0 0" xyz="0.014491 0.136188 -0.024125"/>
+    <inertia ixx="0.000285" ixy="-0.0" ixz="-0.0" iyy="0.000502" iyz="-0.0" izz="0.000285"/>
+  </inertial>
+  <visual>
+    <origin rpy="0 0 0" xyz="-0.014335 -0.107356 -0.024125"/>
     <geometry>
       <mesh filename="package://ppp90_description/meshes/wheel_Mirror__1.stl" scale="0.001 0.001 0.001"/>
@@ -59,5 +64,5 @@
   </visual>
   <collision>
-    <origin rpy="0 0 0" xyz="0.014491 0.136188 -0.024125"/>
+    <origin rpy="0 0 0" xyz="-0.014335 -0.107356 -0.024125"/>
     <geometry>
       <mesh filename="package://ppp90_description/meshes/wheel_Mirror__1.stl" scale="0.001 0.001 0.001"/>
@@ -67,73 +72,52 @@
 <link name="sonyc_1">
   <inertial>
-    <origin rpy="0 0 0" xyz="0.013000365548618742 -0.010235515019977243 5.0631813087009814e-05"/>
+    <origin rpy="0 0 0" xyz="-0.012999900847315296 0.010235790299775449 5.063181308696818e-05"/>
     <mass value="0.0252883585593009"/>
-    <inertia ixx="1e-06" ixy="0.0" ixz="0.0" iyy="5e-06" iyz="-0.0" izz="5e-06"/>
-  </inertial>
-  <visual>
-    <origin rpy="0 0 0" xyz="0.027494 -0.13623 -0.08983"/>
+    <inertia ixx="1e-06" ixy="0.0" ixz="-0.0" iyy="5e-06" iyz="0.0" izz="5e-06"/>
+  </inertial>
+  <visual>
+    <origin rpy="0 0 0" xyz="-0.027338 0.165062 -0.08983"/>
     <geometry>
       <box size="0.001 0.0005 0.00035"/>
-      <!-- <mesh filename="package://ppp90_description/meshes/sonyc_1.stl" scale="0.001 0.001 0.001"/> -->
-    </geometry>
-    <material name="silver"/>
-  </visual>
-  <!-- <collision>
-    <origin rpy="0 0 0" xyz="0.027494 -0.13623 -0.08983"/>
-    <geometry>
-      <mesh filename="package://ppp90_description/meshes/sonyc_1.stl" scale="0.001 0.001 0.001"/>
-    </geometry>
-  </collision> -->
+    </geometry>
+    <material name="silver"/>
+  </visual>
 </link>
 <link name="sonyc_Mirror__1">
   <inertial>
-    <origin rpy="0 0 0" xyz="-0.012999634451381028 0.010235325598471623 5.063181308698206e-05"/>
+    <origin rpy="0 0 0" xyz="0.013000099152684503 -0.010236050318673445 5.063181308696818e-05"/>
     <mass value="0.025288358559300887"/>
-    <inertia ixx="1e-06" ixy="-0.0" ixz="0.0" iyy="5e-06" iyz="0.0" izz="5e-06"/>
-  </inertial>
-  <visual>
-    <origin rpy="0 0 0" xyz="0.001494 0.164906 -0.08983"/>
+    <inertia ixx="1e-06" ixy="-0.0" ixz="-0.0" iyy="5e-06" iyz="-0.0" izz="5e-06"/>
+  </inertial>
+  <visual>
+    <origin rpy="0 0 0" xyz="-0.001338 -0.136075 -0.08983"/>
     <geometry>
       <box size="0.001 0.0005 0.00035"/>
-      <!-- <mesh filename="package://ppp90_description/meshes/sonyc_Mirror__1.stl" scale="0.001 0.001 0.001"/> -->
-    </geometry>
-    <material name="silver"/>
-  </visual>
-  <!-- <collision>
-    <origin rpy="0 0 0" xyz="0.001494 0.164906 -0.08983"/>
-    <geometry>
-      <mesh filename="package://ppp90_description/meshes/sonyc_Mirror__1.stl" scale="0.001 0.001 0.001"/>
-    </geometry>
-  </collision> -->
+    </geometry>
+    <material name="silver"/>
+  </visual>
 </link>
 <link name="sonyc__1__1">
   <inertial>
-    <origin rpy="0 0 0" xyz="0.010235448068739439 -0.013000419106913505 5.063181308698206e-05"/>
+    <origin rpy="0 0 0" xyz="-0.010235983367435975 0.012999694386711707 5.06318130869543e-05"/>
     <mass value="0.0252883585593009"/>
-    <inertia ixx="5e-06" ixy="-0.0" ixz="0.0" iyy="1e-06" iyz="0.0" izz="5e-06"/>
-  </inertial>
-  <visual>
-    <origin rpy="0 0 0" xyz="0.169414 0.001361 -0.06983"/>
+    <inertia ixx="5e-06" ixy="-0.0" ixz="-0.0" iyy="1e-06" iyz="-0.0" izz="5e-06"/>
+  </inertial>
+  <visual>
+    <origin rpy="0 0 0" xyz="-0.169259 0.02747 -0.06983"/>
     <geometry>
       <box size="0.001 0.0005 0.00035"/>
-      <!-- <mesh filename="package://ppp90_description/meshes/sonyc__1__1.stl" scale="0.001 0.001 0.001"/> -->
-    </geometry>
-    <material name="silver"/>
-  </visual>
-  <!-- <collision>
-    <origin rpy="0 0 0" xyz="0.169414 0.001361 -0.06983"/>
-    <geometry>
-      <mesh filename="package://ppp90_description/meshes/sonyc__1__1.stl" scale="0.001 0.001 0.001"/>
-    </geometry>
-  </collision> -->
+    </geometry>
+    <material name="silver"/>
+  </visual>
 </link>
 <link name="nema17_1">
   <inertial>
-    <origin rpy="0 0 0" xyz="-6.709208478471174e-07 -0.00334258185473002 0.02118013525930306"/>
+    <origin rpy="0 0 0" xyz="1.1356221513089682e-06 0.0033428571345282126 0.021180135259303026"/>
     <mass value="0.1838412954712099"/>
-    <inertia ixx="5.2e-05" ixy="-0.0" ixz="-0.0" iyy="5.3e-05" iyz="0.0" izz="5.2e-05"/>
-  </inertial>
-  <visual>
-    <origin rpy="0 0 0" xyz="0.014494 -0.084071 -0.003"/>
+    <inertia ixx="5.2e-05" ixy="-0.0" ixz="0.0" iyy="5.3e-05" iyz="-0.0" izz="5.2e-05"/>
+  </inertial>
+  <visual>
+    <origin rpy="0 0 0" xyz="-0.014338 0.112903 -0.003"/>
     <geometry>
       <mesh filename="package://ppp90_description/meshes/nema17_1.stl" scale="0.001 0.001 0.001"/>
@@ -142,5 +126,5 @@
   </visual>
   <collision>
-    <origin rpy="0 0 0" xyz="0.014494 -0.084071 -0.003"/>
+    <origin rpy="0 0 0" xyz="-0.014338 0.112903 -0.003"/>
     <geometry>
       <mesh filename="package://ppp90_description/meshes/nema17_1.stl" scale="0.001 0.001 0.001"/>
@@ -150,10 +134,10 @@
 <link name="nema17_Mirror__1">
   <inertial>
-    <origin rpy="0 0 0" xyz="-5.975012162888829e-06 0.00334264208445903 0.02118013525930306"/>
+    <origin rpy="0 0 0" xyz="6.439713466371497e-06 -0.003342366804660879 0.021180135259303026"/>
     <mass value="0.1838412954712099"/>
-    <inertia ixx="5.2e-05" ixy="-0.0" ixz="-0.0" iyy="5.3e-05" iyz="-0.0" izz="5.2e-05"/>
-  </inertial>
-  <visual>
-    <origin rpy="0 0 0" xyz="0.014528 0.113338 -0.003"/>
+    <inertia ixx="5.2e-05" ixy="-0.0" ixz="0.0" iyy="5.3e-05" iyz="0.0" izz="5.2e-05"/>
+  </inertial>
+  <visual>
+    <origin rpy="0 0 0" xyz="-0.014372 -0.084506 -0.003"/>
     <geometry>
       <mesh filename="package://ppp90_description/meshes/nema17_Mirror__1.stl" scale="0.001 0.001 0.001"/>
@@ -162,5 +146,5 @@
   </visual>
   <collision>
-    <origin rpy="0 0 0" xyz="0.014528 0.113338 -0.003"/>
+    <origin rpy="0 0 0" xyz="-0.014372 -0.084506 -0.003"/>
     <geometry>
       <mesh filename="package://ppp90_description/meshes/nema17_Mirror__1.stl" scale="0.001 0.001 0.001"/>
@@ -170,10 +154,10 @@
 <link name="12GAN20__1__1">
   <inertial>
-    <origin rpy="0 0 0" xyz="3.268980405812805e-08 -3.387342204674848e-06 0.011857871337072723"/>
+    <origin rpy="0 0 0" xyz="-5.679885005938079e-07 2.662622002880255e-06 0.011857871337072685"/>
     <mass value="0.023492103087793172"/>
-    <inertia ixx="1e-06" ixy="-0.0" ixz="-0.0" iyy="2e-06" iyz="-0.0" izz="0.0"/>
-  </inertial>
-  <visual>
-    <origin rpy="0 0 0" xyz="0.096453 0.12774 -0.001"/>
+    <inertia ixx="1e-06" ixy="-0.0" ixz="0.0" iyy="2e-06" iyz="0.0" izz="0.0"/>
+  </inertial>
+  <visual>
+    <origin rpy="0 0 0" xyz="-0.096298 -0.098909 -0.001"/>
     <geometry>
       <mesh filename="package://ppp90_description/meshes/12GAN20__1__1.stl" scale="0.001 0.001 0.001"/>
@@ -182,5 +166,5 @@
   </visual>
   <collision>
-    <origin rpy="0 0 0" xyz="0.096453 0.12774 -0.001"/>
+    <origin rpy="0 0 0" xyz="-0.096298 -0.098909 -0.001"/>
     <geometry>
       <mesh filename="package://ppp90_description/meshes/12GAN20__1__1.stl" scale="0.001 0.001 0.001"/>
@@ -190,10 +174,10 @@
 <link name="brush_1">
   <inertial>
-    <origin rpy="0 0 0" xyz="-6.629561645765669e-07 -8.680417363238213e-07 -0.0022204199308318013"/>
+    <origin rpy="0 0 0" xyz="1.2765746805476486e-07 1.4332153454310603e-07 -0.0022204199308318365"/>
     <mass value="0.014937067448072668"/>
-    <inertia ixx="1e-06" ixy="0.0" ixz="0.0" iyy="1e-06" iyz="0.0" izz="2e-06"/>
-  </inertial>
-  <visual>
-    <origin rpy="0 0 0" xyz="0.096455 0.12775 0.001"/>
+    <inertia ixx="1e-06" ixy="0.0" ixz="-0.0" iyy="1e-06" iyz="-0.0" izz="2e-06"/>
+  </inertial>
+  <visual>
+    <origin rpy="0 0 0" xyz="-0.0963 -0.098919 0.001"/>
     <geometry>
       <mesh filename="package://ppp90_description/meshes/brush_1.stl" scale="0.001 0.001 0.001"/>
@@ -202,5 +186,5 @@
   </visual>
   <collision>
-    <origin rpy="0 0 0" xyz="0.096455 0.12775 0.001"/>
+    <origin rpy="0 0 0" xyz="-0.0963 -0.098919 0.001"/>
     <geometry>
       <mesh filename="package://ppp90_description/meshes/brush_1.stl" scale="0.001 0.001 0.001"/>
@@ -210,10 +194,10 @@
 <link name="brush_Mirror__1">
   <inertial>
-    <origin rpy="0 0 0" xyz="5.998655124295205e-07 3.438472244571278e-07 -0.0022204199308317827"/>
+    <origin rpy="0 0 0" xyz="-1.1351642089096892e-06 -6.856742623684298e-08 -0.0022204199308317827"/>
     <mass value="0.014937067448072664"/>
-    <inertia ixx="1e-06" ixy="0.0" ixz="-0.0" iyy="1e-06" iyz="0.0" izz="2e-06"/>
-  </inertial>
-  <visual>
-    <origin rpy="0 0 0" xyz="0.096451 -0.099054 0.001"/>
+    <inertia ixx="1e-06" ixy="0.0" ixz="0.0" iyy="1e-06" iyz="-0.0" izz="2e-06"/>
+  </inertial>
+  <visual>
+    <origin rpy="0 0 0" xyz="-0.096296 0.127886 0.001"/>
     <geometry>
       <mesh filename="package://ppp90_description/meshes/brush_Mirror__1.stl" scale="0.001 0.001 0.001"/>
@@ -222,5 +206,5 @@
   </visual>
   <collision>
-    <origin rpy="0 0 0" xyz="0.096451 -0.099054 0.001"/>
+    <origin rpy="0 0 0" xyz="-0.096296 0.127886 0.001"/>
     <geometry>
       <mesh filename="package://ppp90_description/meshes/brush_Mirror__1.stl" scale="0.001 0.001 0.001"/>
@@ -230,10 +214,10 @@
 <link name="12GAN20__1__Mirror__1">
   <inertial>
-    <origin rpy="0 0 0" xyz="2.061205277625877e-06 -6.450130101642859e-06 0.011857871337072723"/>
+    <origin rpy="0 0 0" xyz="-2.596503974161557e-06 6.725409899849266e-06 0.011857871337072688"/>
     <mass value="0.02349210308779317"/>
-    <inertia ixx="1e-06" ixy="0.0" ixz="-0.0" iyy="2e-06" iyz="0.0" izz="0.0"/>
-  </inertial>
-  <visual>
-    <origin rpy="0 0 0" xyz="0.096451 -0.099054 -0.001"/>
+    <inertia ixx="1e-06" ixy="0.0" ixz="0.0" iyy="2e-06" iyz="-0.0" izz="0.0"/>
+  </inertial>
+  <visual>
+    <origin rpy="0 0 0" xyz="-0.096296 0.127886 -0.001"/>
     <geometry>
       <mesh filename="package://ppp90_description/meshes/12GAN20__1__Mirror__1.stl" scale="0.001 0.001 0.001"/>
@@ -242,5 +226,5 @@
   </visual>
   <collision>
-    <origin rpy="0 0 0" xyz="0.096451 -0.099054 -0.001"/>
+    <origin rpy="0 0 0" xyz="-0.096296 0.127886 -0.001"/>
     <geometry>
       <mesh filename="package://ppp90_description/meshes/12GAN20__1__Mirror__1.stl" scale="0.001 0.001 0.001"/>
@@ -248,22 +232,142 @@
   </collision>
 </link>
+<link name="forward_top_1_1">
+  <inertial>
+    <origin rpy="0 0 0" xyz="-0.09472371095209488 -0.06502162145818441 0.0004895173930853369"/>
+    <mass value="0.48710215659029577"/>
+    <inertia ixx="0.000784" ixy="-0.000235" ixz="-1e-06" iyy="0.00099" iyz="-1e-06" izz="0.001773"/>
+  </inertial>
+  <visual>
+    <origin rpy="0 0 0" xyz="-0.163338 0.014494 -0.11"/>
+    <geometry>
+      <mesh filename="package://ppp90_description/meshes/forward_top_1_1.stl" scale="0.001 0.001 0.001"/>
+    </geometry>
+    <material name="silver"/>
+  </visual>
+  <collision>
+    <origin rpy="0 0 0" xyz="-0.163338 0.014494 -0.11"/>
+    <geometry>
+      <mesh filename="package://ppp90_description/meshes/forward_top_1_1.stl" scale="0.001 0.001 0.001"/>
+    </geometry>
+  </collision>
+</link>
+<link name="forward_top_1_Mirror__1">
+  <inertial>
+    <origin rpy="0 0 0" xyz="0.0735909092846742 -0.07845842785085694 0.0004895171912021601"/>
+    <mass value="0.48710223650351714"/>
+    <inertia ixx="0.000784" ixy="0.000234" ixz="-1e-06" iyy="0.00099" iyz="1e-06" izz="0.001773"/>
+  </inertial>
+  <visual>
+    <origin rpy="0 0 0" xyz="0.005021 -0.129037 -0.11"/>
+    <geometry>
+      <mesh filename="package://ppp90_description/meshes/forward_top_1_Mirror__1.stl" scale="0.001 0.001 0.001"/>
+    </geometry>
+    <material name="silver"/>
+  </visual>
+  <collision>
+    <origin rpy="0 0 0" xyz="0.005021 -0.129037 -0.11"/>
+    <geometry>
+      <mesh filename="package://ppp90_description/meshes/forward_top_1_Mirror__1.stl" scale="0.001 0.001 0.001"/>
+    </geometry>
+  </collision>
+</link>
+<link name="back_top_1">
+  <inertial>
+    <origin rpy="0 0 0" xyz="-0.06983924477939416 -0.07365384534784823 -0.0010887199497685157"/>
+    <mass value="0.23560428740017997"/>
+    <inertia ixx="0.000537" ixy="-0.000345" ixz="-1.3e-05" iyy="0.00038" iyz="-1.8e-05" izz="0.000907"/>
+  </inertial>
+  <visual>
+    <origin rpy="0 0 0" xyz="0.005021 -0.129037 -0.11"/>
+    <geometry>
+      <mesh filename="package://ppp90_description/meshes/back_top_1.stl" scale="0.001 0.001 0.001"/>
+    </geometry>
+    <material name="silver"/>
+  </visual>
+  <collision>
+    <origin rpy="0 0 0" xyz="0.005021 -0.129037 -0.11"/>
+    <geometry>
+      <mesh filename="package://ppp90_description/meshes/back_top_1.stl" scale="0.001 0.001 0.001"/>
+    </geometry>
+  </collision>
+</link>
+<link name="back_top2_1">
+  <inertial>
+    <origin rpy="0 0 0" xyz="-0.05870936689603044 0.05499707718659973 0.0004968868769272966"/>
+    <mass value="0.18961170684744505"/>
+    <inertia ixx="0.000183" ixy="0.000153" ixz="1e-06" iyy="0.000249" iyz="-1e-06" izz="0.000432"/>
+  </inertial>
+  <visual>
+    <origin rpy="0 0 0" xyz="0.005021 0.158024 -0.11"/>
+    <geometry>
+      <mesh filename="package://ppp90_description/meshes/back_top2_1.stl" scale="0.001 0.001 0.001"/>
+    </geometry>
+    <material name="silver"/>
+  </visual>
+  <collision>
+    <origin rpy="0 0 0" xyz="0.005021 0.158024 -0.11"/>
+    <geometry>
+      <mesh filename="package://ppp90_description/meshes/back_top2_1.stl" scale="0.001 0.001 0.001"/>
+    </geometry>
+  </collision>
+</link>
+<link name="Lidar_1">
+  <inertial>
+    <origin rpy="0 0 0" xyz="3.0855486037040247e-07 2.620424081334338e-07 0.03500000000000002"/>
+    <mass value="2.114723824855799"/>
+    <inertia ixx="0.001511" ixy="-0.0" ixz="-0.0" iyy="0.001511" iyz="0.0" izz="0.001295"/>
+  </inertial>
+  <visual>
+    <origin rpy="0 0 0" xyz="-0.110658 0.014415 -0.112"/>
+    <geometry>
+      <mesh filename="package://ppp90_description/meshes/Lidar_1.stl" scale="0.001 0.001 0.001"/>
+    </geometry>
+    <material name="silver"/>
+  </visual>
+  <collision>
+    <origin rpy="0 0 0" xyz="-0.110658 0.014415 -0.112"/>
+    <geometry>
+      <mesh filename="package://ppp90_description/meshes/Lidar_1.stl" scale="0.001 0.001 0.001"/>
+    </geometry>
+  </collision>
+</link>
+<link name="IMU_1">
+  <inertial>
+    <origin rpy="0 0 0" xyz="-1.0482840423486905e-07 3.699905506693302e-07 0.007500000000000007"/>
+    <mass value="0.011774999999999999"/>
+    <inertia ixx="1e-06" ixy="0.0" ixz="0.0" iyy="0.0" iyz="-0.0" izz="0.0"/>
+  </inertial>
+  <visual>
+    <origin rpy="0 0 0" xyz="-0.158919 0.014494 -0.033"/>
+    <geometry>
+      <mesh filename="package://ppp90_description/meshes/IMU_1.stl" scale="0.001 0.001 0.001"/>
+    </geometry>
+    <material name="silver"/>
+  </visual>
+  <collision>
+    <origin rpy="0 0 0" xyz="-0.158919 0.014494 -0.033"/>
+    <geometry>
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
Commit message: hz1

File: src/ppp90_description/urdf/ppp90.xacro (robot description, xacro)
@@ -399,5 +399,5 @@
     <inertia ixx="1e-06" ixy="0.0" ixz="0.0" iyy="0.0" iyz="0.0" izz="1e-06"/>
   </inertial>
-  <visual>
+  <visual><!---0.0175 -0.015 0-->
     <origin rpy="0 0 0" xyz="0.053573 -0.022977 -0.0025"/>
     <geometry>
@@ -420,5 +420,5 @@
   </inertial>
   <visual>
-    <origin rpy="0 0 0" xyz="-0.0175 -0.015 0.0"/>
+    <origin rpy="0 0 0" xyz="-0.0054 -0.104 -0.015"/>
     <geometry>
       <mesh filename="package://ppp90_description/meshes/holder2_1.stl" scale="0.001 0.001 0.001"/>
@@ -459,5 +459,5 @@
 </joint>
 <joint name="Rev11" type="continuous">
-  <origin rpy="0 0 0" xyz="0.0 0.0 0.0"/>
+  <origin rpy="0 0 0" xyz="0.0 0.015 0.0"/>
   <parent link="fww_a_1"/>
   <child link="fw_wheel_1"/>
@@ -465,5 +465,5 @@
 </joint>
 <joint name="Rev21" type="continuous">
-  <origin rpy="0 0 0" xyz="-0.071073 0.007977 0.0025"/>
+  <origin rpy="0 0 0" xyz="0 0 0"/>
   <parent link="holder2_1"/>
   <child link="holder1_1"/>
@@ -477,5 +477,5 @@
 </joint>
 <joint name="Rev41" type="continuous">
-  <origin rpy="0 0 0" xyz="0 0 0"/>
+  <origin rpy="0 0 0" xyz="0.028684 -0.031977 0.03341"/>
   <parent link="holder1_1"/>
   <child link="fww_a_1"/>
