Commit message: ball

File: src/ppp90_description/urdf/ppp90.xacro (robot description, xacro)
@@ -334,5 +334,5 @@
 <link name="IMU_1">
   <inertial>
-    <origin rpy="0 0 0" xyz="-1.0482840423486905e-07 3.699905506693302e-07 0.007500000000000007"/>
+    <origin rpy="0 0 0" xyz="-0.158919 0.014494 -0.033"/>
     <mass value="0.011774999999999999"/>
     <inertia ixx="1e-06" ixy="0.0" ixz="0.0" iyy="0.0" iyz="-0.0" izz="0.0"/>
@@ -353,133 +353,27 @@
 </link>
 <!-- -->
-<link name="Forward_wheel_1">
-  <inertial>
-    <origin rpy="0 0 0" xyz="-0.120769 0.014494 -0.022"/>
-    <mass value="0.0061871055650105375"/>
-    <inertia ixx="0.0" ixy="0.0" ixz="-0.0" iyy="0.0" iyz="-0.0" izz="1e-06"/>
-  </inertial>
-  <visual>
-    <origin rpy="0 0 0" xyz="-0.120769 0.014494 -0.022"/>
-    <geometry>
-      <mesh filename="package://ppp90_description/meshes/Forward_wheel_1.stl" scale="0.001 0.001 0.001"/>
-    </geometry>
-    <material name="silver"/>
-  </visual>
-  <collision>
-    <origin rpy="0 0 0" xyz="-0.120769 0.014494 -0.022"/>
-    <geometry>
-      <mesh filename="package://ppp90_description/meshes/Forward_wheel_1.stl" scale="0.001 0.001 0.001"/>
-    </geometry>
-  </collision>
-</link>
-<link name="fw_wheel_1">
-  <inertial>
-    <origin rpy="0 0 0" xyz="0.024889 -0.006 -0.03591"/>
-    <mass value="0.0030764824061019756"/>
-    <inertia ixx="0.0" ixy="-0.0" ixz="0.0" iyy="0.0" iyz="0.0" izz="0.0"/>
-  </inertial>
-  <visual>
-    <origin rpy="0 0 0" xyz="0.024889 -0.006 -0.03591"/>
-    <geometry>
-      <mesh filename="package://ppp90_description/meshes/fw_wheel_1.stl" scale="0.001 0.001 0.001"/>
-    </geometry>
-    <material name="yellow"/>
-  </visual>
-  <collision>
-    <origin rpy="0 0 0" xyz="0.024889 -0.006 -0.03591"/>
-    <geometry>
-      <mesh filename="package://ppp90_description/meshes/fw_wheel_1.stl" scale="0.001 0.001 0.001"/>
-    </geometry>
-  </collision>
-</link>
-<link name="holder1_1">
-  <inertial>
-    <origin rpy="0 0 0" xyz="0.053573 -0.022977 -0.0025"/>
-    <mass value="0.006489971019909515"/>
-    <inertia ixx="1e-06" ixy="0.0" ixz="0.0" iyy="0.0" iyz="0.0" izz="1e-06"/>
-  </inertial>
-  <visual><!---0.0175 -0.015 0-->
-    <origin rpy="0 0 0" xyz="0.053573 -0.022977 -0.0025"/>
-    <geometry>
-      <mesh filename="package://ppp90_description/meshes/holder1_1.stl" scale="0.001 0.001 0.001"/>
-    </geometry>
-    <material name="green"/>
-  </visual>
-  <collision>
-    <origin rpy="0 0 0" xyz="0.053573 -0.022977 -0.0025"/>
-    <geometry>
-      <mesh filename="package://ppp90_description/meshes/holder1_1.stl" scale="0.001 0.001 0.001"/>
-    </geometry>
-  </collision>
-</link>
-<link name="holder2_1">
-  <inertial>
-    <origin rpy="0 0 0" xyz="-0.0175 -0.015 0.0"/>
-    <mass value="0.002767366136694294"/>
-    <inertia ixx="0.0" ixy="0.0" ixz="-0.0" iyy="0.0" iyz="-0.0" izz="0.0"/>
-  </inertial>
-  <visual>
-    <origin rpy="0 0 0" xyz="-0.0054 -0.104 -0.015"/>
-    <geometry>
-      <mesh filename="package://ppp90_description/meshes/holder2_1.stl" scale="0.001 0.001 0.001"/>
-    </geometry>
-    <material name="d_blue"/>
-  </visual>
-  <collision>
-    <origin rpy="0 0 0" xyz="-0.0175 -0.015 0.0"/>
-    <geometry>
-      <mesh filename="package://ppp90_description/meshes/holder2_1.stl" scale="0.001 0.001 0.001"/>
-    </geometry>
-  </collision>
-</link>
-<link name="fww_a_1">
-  <inertial>
-    <origin rpy="0 0 0" xyz="0.0379390477443535 0.11460348542678987 -0.04141447070571836"/>
-    <mass value="0.0043107049436968805"/>
-    <inertia ixx="0.0" ixy="0.0" ixz="0.0" iyy="0.0" iyz="0.0" izz="0.0"/>
-  </inertial>
-  <visual>
-    <origin rpy="0 0 0" xyz="0.024889 0.009 -0.03591"/>
-    <geometry>
-      <mesh filename="package://ppp90_description/meshes/fww_a_1.stl" scale="0.001 0.001 0.001"/>
-    </geometry>
-    <material name="silver"/>
-  </visual>
-  <collision>
-    <origin rpy="0 0 0" xyz="0.024889 0.009 -0.03591"/>
-    <geometry>
-      <mesh filename="package://ppp90_description/meshes/fww_a_1.stl" scale="0.001 0.001 0.001"/>
-    </geometry>
-  </collision>
-</link>
-<joint name="Rigid119" type="fixed">
-  <origin rpy="0 0 0" xyz="0.120769 -0.014494 0.022"/>
-  <parent link="base_link"/>
-  <child link="Forward_wheel_1"/>
-</joint>
-<joint name="Rev11" type="continuous">
-  <origin rpy="0 0 0" xyz="0.0 0.015 0.0"/>
-  <parent link="fww_a_1"/>
-  <child link="fw_wheel_1"/>
-  <axis xyz="-0.258819 0.965926 0.0"/>
-</joint>
-<joint name="Rev21" type="continuous">
-  <origin rpy="0 0 0" xyz="0 0 0"/>
-  <parent link="holder2_1"/>
-  <child link="holder1_1"/>
-  <axis xyz="-0.0 0.0 -1.0"/>
-</joint>
-<joint name="Rev31" type="continuous">
-  <origin rpy="0 0 0" xyz="0 0 0"/>
-  <parent link="Forward_wheel_1"/>
-  <child link="holder2_1"/>
-  <axis xyz="0.0 -0.0 1.0"/>
-</joint>
-<joint name="Rev41" type="continuous">
-  <origin rpy="0 0 0" xyz="0.028684 -0.031977 0.03341"/>
-  <parent link="holder1_1"/>
-  <child link="fww_a_1"/>
-  <axis xyz="0.258819 -0.965926 -0.0"/>
-</joint>
+    <link name='link_1'>
+      <inertial>
+        <mass value="0.3" />
+        <origin xyz="0 0 0" />
+        <inertia  ixx="1.0" ixy="0.0"  ixz="0.0"  iyy="1.0"  iyz="0.0"  izz="1.0" />
+      </inertial>
+      <visual>
+        <origin xyz="0.12116 -0.014724 0.1499" rpy="0 0 0" />
+        <geometry>
+          <sphere radius="0.0215773"/>
+        </geometry>
+      </visual>
+      <collision>
+        <origin xyz="0 0 0" rpy="0 0 0" />
+        <geometry>
+          <sphere radius="0.0215773"/>
+        </geometry>
+      </collision>
+    </link>
+    <joint name='base_footprint_JOINT_2' type='continuous'>
+       <parent link="base_link"/>
+       <child link="link_1"/>
+    </joint>
 <!-- -->
 <joint name="Rev1" type="continuous">

Commit message: ebaniy urdf

File: src/ppp90_description/urdf/ppp90.xacro (robot description, xacro)
@@ -12,10 +12,10 @@
 <link name="base_link">
   <inertial>
-    <origin rpy="0 0 0" xyz="0.006228517780792832 -0.014312684450430895 0.03416379967065732"/>
+    <origin rpy="0 0 1.5708" xyz="0 0 0"/>
     <mass value="5.029311101542255"/>
     <inertia ixx="0.037081" ixy="0.000111" ixz="0.001835" iyy="0.04462" iyz="-2e-05" izz="0.070617"/>
   </inertial>
   <visual>
-    <origin rpy="0 0 0" xyz="0 0 0"/>
+    <origin rpy="0 0 1.5708" xyz="0 0 0"/>
     <geometry>
       <mesh filename="package://ppp90_description/meshes/base_link.stl" scale="0.001 0.001 0.001"/>
@@ -24,5 +24,5 @@
   </visual>
   <collision>
-    <origin rpy="0 0 0" xyz="0 0 0"/>
+    <origin rpy="0 0 1.5708" xyz="0 0 0"/>
     <geometry>
       <mesh filename="package://ppp90_description/meshes/base_link.stl" scale="0.001 0.001 0.001"/>

File: src/ppp_description/urdf/ppp.xacro (robot description, xacro)
@@ -4,4 +4,10 @@
 <xacro:include filename="$(find ppp_description)/urdf/ppp.trans" />
 <xacro:include filename="$(find ppp_description)/urdf/ppp.gazebo" />
+<link name="base_footprint"/>
+<joint name="base_joint" type="fixed">
+    <parent link="base_footprint"/>
+    <child link="base_link"/>
+    <origin xyz="0.0 0.0 0.010" rpy="0 0 0"/>
+</joint>
 <link name="base_link">
   <inertial><!--1.5708-->

Commit message: fix lidar

File: src/ppp90_description/urdf/ppp90.xacro (robot description, xacro)
@@ -12,10 +12,10 @@
 <link name="base_link">
   <inertial>
-    <origin rpy="0 0 1.5708" xyz="0 0 0"/>
+    <origin rpy="0 0 0" xyz="0 0 0"/>
     <mass value="5.029311101542255"/>
     <inertia ixx="0.037081" ixy="0.000111" ixz="0.001835" iyy="0.04462" iyz="-2e-05" izz="0.070617"/>
   </inertial>
   <visual>
-    <origin rpy="0 0 1.5708" xyz="0 0 0"/>
+    <origin rpy="0 0 0" xyz="0 0 0"/>
     <geometry>
       <mesh filename="package://ppp90_description/meshes/base_link.stl" scale="0.001 0.001 0.001"/>
@@ -24,5 +24,5 @@
   </visual>
   <collision>
-    <origin rpy="0 0 1.5708" xyz="0 0 0"/>
+    <origin rpy="0 0 0" xyz="0 0 0"/>
     <geometry>
       <mesh filename="package://ppp90_description/meshes/base_link.stl" scale="0.001 0.001 0.001"/>
@@ -457,5 +457,5 @@
 </joint>
 <joint name="Rigid25" type="fixed">
-  <origin rpy="0 0 0" xyz="0.115679 -0.143452 0.002"/>
+  <origin rpy="0 0 3.14159" xyz="0.115679 -0.143452 0.002"/>
   <parent link="forward_top_1_Mirror__1"/>
   <child link="Lidar_1"/>

Commit message: fix some params

File: src/ppp90_description/urdf/ppp90.xacro (robot description, xacro)
@@ -332,5 +332,5 @@
   </collision>
 </link>
-<link name="IMU_1">
+<link name="base_imu_link">
   <inertial>
     <origin rpy="0 0 0" xyz="-0.158919 0.014494 -0.033"/>
@@ -464,5 +464,5 @@
   <origin rpy="0 0 0" xyz="0.158919 -0.014494 0.033"/>
   <parent link="base_link"/>
-  <child link="IMU_1"/>
+  <child link="base_imu_link"/>
 </joint>
 </robot>

Commit message: 50/50 gazebo

File: src/ppp90_description/urdf/ppp90.xacro (robot description, xacro)
@@ -353,27 +353,28 @@
 </link>
 <!-- -->
-    <link name='link_1'>
-      <inertial>
-        <mass value="0.3" />
-        <origin xyz="0 0 0" />
-        <inertia  ixx="1.0" ixy="0.0"  ixz="0.0"  iyy="1.0"  iyz="0.0"  izz="1.0" />
-      </inertial>
-      <visual>
-        <origin xyz="0.12116 -0.014724 0.1499" rpy="0 0 0" />
-        <geometry>
-          <sphere radius="0.0215773"/>
-        </geometry>
-      </visual>
-      <collision>
-        <origin xyz="0 0 0" rpy="0 0 0" />
-        <geometry>
-          <sphere radius="0.0215773"/>
-        </geometry>
-      </collision>
-    </link>
-    <joint name='base_footprint_JOINT_2' type='continuous'>
-       <parent link="base_link"/>
-       <child link="link_1"/>
-    </joint>
+  <link name='link_1'>
+    <inertial>
+      <origin xyz="0 0 0" rpy="0 0 0" />
+      <mass value="0.3" />
+      <inertia ixx="1e-06" ixy="0.0" ixz="0.0" iyy="0.0" iyz="-0.0" izz="0.0"/>
+    </inertial>
+    <visual>
+      <origin xyz="0 0 0" rpy="0 0 0" />
+      <geometry>
+        <sphere radius="0.0215773"/>
+      </geometry>
+    </visual>
+    <collision>
+      <origin xyz="0 0 0" rpy="0 0 0" />
+      <geometry>
+        <sphere radius="0.0215773"/>
+      </geometry>
+    </collision>
+  </link>
+  <joint name='base_footprint_JOINT_2' type='continuous'>
+      <origin xyz="0.12116 -0.014724 0.01" rpy="0 0 0" />
+      <parent link="base_link"/>
+      <child link="link_1"/>
+  </joint>
 <!-- -->
 <joint name="Rev1" type="continuous">

Commit message: fix sonic position

File: src/ppp90_description/urdf/ppp90.xacro (robot description, xacro)
@@ -391,10 +391,10 @@
 </joint>
 <joint name="Rigid5" type="fixed">
-  <origin rpy="0 0 0" xyz="0.027338 -0.165062 0.08983"/>
+  <origin rpy="0 0 -1.5708" xyz="0.027338 -0.165062 0.08983"/>
   <parent link="base_link"/>
   <child link="sonyc_1"/>
 </joint>
 <joint name="Rigid6" type="fixed">
-  <origin rpy="0 0 0" xyz="0.001338 0.136075 0.08983"/>
+  <origin rpy="0 0 1.5708" xyz="0.001338 0.136075 0.08983"/>
   <parent link="base_link"/>
   <child link="sonyc_Mirror__1"/>

Commit message: fix gazebo OK!!!

File: src/ppp90_description/urdf/ppp90.xacro (robot description, xacro)
@@ -29,4 +29,26 @@
     </geometry>
   </collision>
+  <visual name="caster_front_visual">
+    <origin xyz="0.12116 -0.014724 0.01" rpy="0 0 0" />
+    <geometry>
+      <sphere radius="0.0215773"/>
+    </geometry>
+    <surface>
+      <friction>
+        <ode>
+          <mu>0</mu>
+          <mu2>0</mu2>
+          <slip1>1.0</slip1>
+          <slip2>1.0</slip2>
+        </ode>
+      </friction>
+    </surface>
+  </visual>
+  <collision name="caster_front_collision">
+    <origin xyz="0.12116 -0.014724 0.01" rpy="0 0 0" />
+    <geometry>
+      <sphere radius="0.0215773"/>
+    </geometry>
+  </collision>
 </link>
 <link name="wheel_1">
@@ -353,5 +375,5 @@
 </link>
 <!-- -->
-  <link name='link_1'>
+  <!-- <link name='link_1'>
     <inertial>
       <origin xyz="0 0 0" rpy="0 0 0" />
@@ -376,5 +398,5 @@
       <parent link="base_link"/>
       <child link="link_1"/>
-  </joint>
+  </joint> -->
 <!-- -->
 <joint name="Rev1" type="continuous">

Commit message: test ball, in progress

File: src/ppp90_description/urdf/ppp90.xacro (robot description, xacro)
@@ -29,8 +29,41 @@
     </geometry>
   </collision>
-  <visual name="caster_front_visual">
-    <origin xyz="0.12116 -0.014724 0.01" rpy="0 0 0" />
-    <geometry>
-      <sphere radius="0.0215773"/>
+</link>
+<link name="roll_celinder">
+    <inertial>
+      <origin  xyz="0 0 0" rpy="0 0 0"/>
+      <mass value="0.1"/>
+      <inertia ixx="0.000285" ixy="-0.0" ixz="-0.0" iyy="0.000502" iyz="-0.0" izz="0.000285"/>
+    </inertial>
+    <visual>
+        <origin rpy="0 0 0" xyz="0 0 0"/>
+        <geometry>
+            <cylinder length="0.005" radius="0.01"/>
+        </geometry>
+        <material name="red"/>
+    </visual>
+      <collision>
+    <origin xyz="0 0 0" rpy="0 0 0" />
+    <geometry>
+       <cylinder length="0.005" radius="0.01"/>
+    </geometry>
+  </collision>
+</link>
+<joint name="celinder_celinder" type="continuous">
+  <origin  xyz="0.12116 -0.014724 -0.001" rpy="0 0 0"/>
+  <parent link="base_link"/>
+  <child link="roll_celinder"/>
+  <axis xyz="-0 -0.0 -1.0"/>
+</joint>
+<link name="ball">
+  <inertial>
+    <origin  xyz="0 0 0" rpy="0 0 0"/>
+    <mass value="4"/>
+    <inertia ixx="0.000285" ixy="-0.0" ixz="-0.0" iyy="0.000502" iyz="-0.0" izz="0.000285"/>
+  </inertial>
+  <visual >
+    <origin xyz="0 0 0" rpy="0 0 0" />
+    <geometry>
+      <sphere radius="0.01"/>
     </geometry>
     <surface>
@@ -45,11 +78,17 @@
     </surface>
   </visual>
-  <collision name="caster_front_collision">
-    <origin xyz="0.12116 -0.014724 0.01" rpy="0 0 0" />
-    <geometry>
-      <sphere radius="0.0215773"/>
-    </geometry>
-  </collision>
-</link>
+  <collision>
+    <origin xyz="0 0 0" rpy="0 0 0" />
+    <geometry>
+      <sphere radius="0.01"/>
+    </geometry>
+  </collision>
+</link>
+<joint name="b_ball" type="continuous">
+  <origin  xyz="0.0 -0.0 -0.001" rpy="0 0 0"/>
+  <parent link="roll_celinder"/>
+  <child link="ball"/>
+  <axis xyz="0.0 -1.0 -0.0"/>
+</joint>
 <link name="wheel_1">
   <inertial>
@@ -401,5 +440,5 @@
 <!-- -->
 <joint name="Rev1" type="continuous">
-  <origin rpy="0 0 0" xyz="0.0 -0.04585 0.021125"/>
+  <origin rpy="3.14159 0 0" xyz="0.0 -0.025 0.021125"/>
   <parent link="nema17_1"/>
   <child link="wheel_1"/>

Commit message: urdf ok

File: src/ppp90_description/urdf/ppp90.xacro (robot description, xacro)
@@ -381,5 +381,5 @@
   </collision>
 </link>
-<link name="Lidar_1">
+<link name="Lidar_Box">
   <inertial>
     <origin rpy="0 0 0" xyz="3.0855486037040247e-07 2.620424081334338e-07 0.03500000000000002"/>
@@ -401,4 +401,35 @@
   </collision>
 </link>
+<link name="Lidar_1">
+  <inertial>
+    <origin rpy="0 0 0" xyz="0 0 0"/>
+    <mass value="0.001"/>
+    <inertia ixx="0.001511" ixy="-0.0" ixz="-0.0" iyy="0.001511" iyz="0.0" izz="0.001295"/>
+  </inertial>
+  <visual>
+    <origin rpy="0 0 0" xyz="0 0 0"/>
+    <geometry>
+      <cylinder length="0.02" radius="0.02"/>
+    </geometry>
+    <material name="red"/>
+  </visual>
+  <collision>
+    <origin rpy="0 0 0" xyz="0 0 0"/>
+    <geometry>
+      <cylinder length="0.02" radius="0.02"/>
+    </geometry>
+  </collision>
+</link>
+<joint name="Lidar_box_to_base_link" type="fixed">
+  <origin rpy="0 0 3.14159" xyz="0.115679 -0.143452 0.002"/>
+  <parent link="forward_top_1_Mirror__1"/>
+  <child link="Lidar_Box"/>
+</joint>
+<joint name="Lidar_Box_LIDAR" type="fixed">
+  <origin rpy="3.14159 0 0" xyz="0.0 0 0.07"/>
+  <parent link="Lidar_Box"/>
+  <child link="Lidar_1"/>
+  <axis xyz="0.0 -1.0 -0.0"/>
+</joint>
 <link name="base_imu_link">
   <inertial>
@@ -421,30 +452,4 @@
   </collision>
 </link>
-<!-- -->
-  <!-- <link name='link_1'>
-    <inertial>
-      <origin xyz="0 0 0" rpy="0 0 0" />
-      <mass value="0.3" />
-      <inertia ixx="1e-06" ixy="0.0" ixz="0.0" iyy="0.0" iyz="-0.0" izz="0.0"/>
-    </inertial>
-    <visual>
-      <origin xyz="0 0 0" rpy="0 0 0" />
-      <geometry>
-        <sphere radius="0.0215773"/>
-      </geometry>
-    </visual>
-    <collision>
-      <origin xyz="0 0 0" rpy="0 0 0" />
-      <geometry>
-        <sphere radius="0.0215773"/>
-      </geometry>
-    </collision>
-  </link>
-  <joint name='base_footprint_JOINT_2' type='continuous'>
-      <origin xyz="0.12116 -0.014724 0.01" rpy="0 0 0" />
-      <parent link="base_link"/>
-      <child link="link_1"/>
-  </joint> -->
-<!-- -->
 <joint name="Rev1" type="continuous">
   <origin rpy="3.14159 0 0" xyz="0.0 -0.025 0.021125"/>
@@ -526,9 +531,4 @@
   <child link="back_top2_1"/>
 </joint>
-<joint name="Rigid25" type="fixed">
-  <origin rpy="0 0 3.14159" xyz="0.115679 -0.143452 0.002"/>
-  <parent link="forward_top_1_Mirror__1"/>
-  <child link="Lidar_1"/>
-</joint>
 <joint name="Rigid26" type="fixed">
   <origin rpy="0 0 0" xyz="0.158919 -0.014494 0.033"/>

Commit message: turn lidar

File: src/ppp90_description/urdf/ppp90.xacro (robot description, xacro)
@@ -427,5 +427,5 @@
 </joint>
 <joint name="Lidar_Box_LIDAR" type="fixed">
-  <origin rpy="3.14159 0 0" xyz="0.0 0 0.07"/>
+  <origin rpy="0 0 3.14159" xyz="0.0 0 0.07"/>
   <parent link="Lidar_Box"/>
   <child link="Lidar_1"/>

Commit message: fucking urdf

File: src/ppp90_description/urdf/ppp90.xacro (robot description, xacro)
@@ -422,5 +422,5 @@
 </link>
 <joint name="Lidar_box_to_base_link" type="fixed">
-  <origin rpy="0 0 3.14159" xyz="0.115679 -0.143452 0.002"/>
+  <origin rpy="0 0 0" xyz="0.115679 -0.143452 0.002"/>
   <parent link="forward_top_1_Mirror__1"/>
   <child link="Lidar_Box"/>
